Commit message: rtab map slam added

File: ros2_rm_robot/dual_rm_description/dual_rm_65b_description/urdf/dual_rm_65b_description.urdf.xacro (robot description, xacro)
@@ -14,4 +14,3 @@
   <xacro:include filename="$(find dual_rm_65b_description)/urdf/body_head_platform_transmission.xacro"/>
   <xacro:include filename="$(find dual_rm_65b_description)/urdf/woosh_agv_transmission.xacro"/>
-  <!-- <xacro:include filename="$(find dual_rm_65b_description)/urdf/common_gazebo.xacro"/> -->
 </robot>

File: ros2_rm_robot/dual_rm_description/dual_rm_65b_description/urdf/woosh_agv_transmission.xacro (robot description, xacro)
@@ -16,14 +16,3 @@
   <xacro:woosh_agv_transmission joint_name="joint_right_wheel" />
   <xacro:woosh_agv_transmission joint_name="joint_left_wheel" />
-  <!-- Optional: Swivel Wheels Transmissions (if you want them controlled) -->
-  <!-- Uncomment these if you need swivel wheels to be controlled by ros2_control -->
-<!--
-  <xacro:woosh_agv_transmission joint_name="joint_swivel_wheel_1_1" />
-  <xacro:woosh_agv_transmission joint_name="joint_swivel_wheel_1_2" />
-  <xacro:woosh_agv_transmission joint_name="joint_swivel_wheel_2_1" />
-  <xacro:woosh_agv_transmission joint_name="joint_swivel_wheel_2_2" />
-  <xacro:woosh_agv_transmission joint_name="joint_swivel_wheel_3_1" />
-  <xacro:woosh_agv_transmission joint_name="joint_swivel_wheel_3_2" />
-  <xacro:woosh_agv_transmission joint_name="joint_swivel_wheel_4_1" />
-  <xacro:woosh_agv_transmission joint_name="joint_swivel_wheel_4_2" /> -->
 </robot>

File: ros2_rm_robot/dual_rm_simulation/dual_rm_65b_gazebo/urdf/depth_camera_65b_gazebo.xacro (robot description, xacro)
@@ -5,5 +5,5 @@
         <sensor name="depth_camera" type="depth">
             <!-- Rotate sensor to match optical frame -->
-            <pose>0 0 0 ${-pi/2} 0 ${-pi/2}</pose>
+            <pose>0.0016556 -0.01252 1.2156E-05 0 0 0</pose>
             <visualize>true</visualize>
             <update_rate>30.0</update_rate>
@@ -29,5 +29,5 @@
         <!-- IMU Sensor (shares same coordinate system as depth sensor) -->
         <sensor name="camera_imu" type="imu">
-            <pose>0 0 0 ${-pi/2} 0 ${-pi/2}</pose>  <!-- Same rotation as camera -->
+            <pose>0.0016556 -0.01252 1.2156E-05 0 0 0</pose>  <!-- Same rotation as camera -->
             <always_on>true</always_on>
             <update_rate>200</update_rate>

File: ros2_rm_robot/dual_rm_simulation/dual_rm_65b_gazebo/urdf/dual_rm_65b_gazebo.urdf.xacro (robot description, xacro)
@@ -1,9 +1,9 @@
 <?xml version="1.0"?>
 <robot xmlns:xacro="http://www.ros.org/wiki/xacro" name="dual_rm_65b_gazebo">
-    <link name="world"/>
-    <joint name="world_to_base_link" type="fixed">
-        <parent link="world"/>
+    <link name="base_footprint"/>
+    <joint name="base_footprint_to_base_link" type="fixed">
+        <parent link="base_footprint"/>
         <child link="base_link_underpan"/>
-        <origin xyz="0 0 0" rpy="0 0 0"/>
+        <origin xyz="0 0 0" rpy="0 0 ${pi/2}"/>
     </joint>
     <xacro:include filename="$(find dual_rm_65b_description)/urdf/dual_rm_65b_description.urdf.xacro" />
@@ -86,41 +86,41 @@
     </gazebo>
     <gazebo reference="link_swivel_wheel_1_1">
-        <mu1 value="0.000002" />
-        <mu2 value="0.000002" />
+        <mu1>0.0005</mu1>
+        <mu2>0.0005</mu2>
         <material>Gazebo/White</material>
     </gazebo>
     <gazebo reference="link_swivel_wheel_1_2">
-        <mu1 value="0.000002" />
-        <mu2 value="0.000002" />
+        <mu1>0.0005</mu1>
+        <mu2>0.0005</mu2>
         <material>Gazebo/White</material>
     </gazebo>
     <gazebo reference="link_swivel_wheel_2_1">
-        <mu1 value="0.000002" />
-        <mu2 value="0.000002" />
+        <mu1>0.0005</mu1>
+        <mu2>0.0005</mu2>
         <material>Gazebo/White</material>
     </gazebo>
     <gazebo reference="link_swivel_wheel_2_2">
-        <mu1 value="0.000002" />
-        <mu2 value="0.000002" />
+        <mu1>0.0005</mu1>
+        <mu2>0.0005</mu2>
         <material>Gazebo/White</material>
     </gazebo>
     <gazebo reference="link_swivel_wheel_3_1">
-        <mu1 value="0.000002" />
-        <mu2 value="0.000002" />
+        <mu1>0.0005</mu1>
+        <mu2>0.0005</mu2>
         <material>Gazebo/White</material>
     </gazebo>
     <gazebo reference="link_swivel_wheel_3_2">
-        <mu1 value="0.000002" />
-        <mu2 value="0.000002" />
+        <mu1>0.0005</mu1>
+        <mu2>0.0005</mu2>
         <material>Gazebo/White</material>
     </gazebo>
     <gazebo reference="link_swivel_wheel_4_1">
-        <mu1 value="0.000002" />
-        <mu2 value="0.000002" />
+        <mu1>0.0005</mu1>
+        <mu2>0.0005</mu2>
         <material>Gazebo/White</material>
     </gazebo>
     <gazebo reference="link_swivel_wheel_4_2">
-        <mu1 value="0.000002" />
-        <mu2 value="0.000002" />
+        <mu1>0.0005</mu1>
+        <mu2>0.0005</mu2>
         <material>Gazebo/White</material>
     </gazebo>

File: ros2_rm_robot/dual_rm_simulation/dual_rm_65b_gazebo/urdf/dual_rm_65b_sim.ros2_control.xacro (robot description, xacro)
@@ -216,5 +216,4 @@
         <!-- Passive Swivel Wheels - No command interface, only state -->
         <joint name="joint_swivel_wheel_1_1">
-            <!-- NO command_interface - this is passive -->
             <state_interface name="position">
                 <param name="initial_value">0</param>
