Commit message: hand joints fixed

File: ros2_rm_robot/dual_rm_description/dual_rm_65b_description/urdf/left_hand.urdf.xacro (robot description, xacro)
@@ -219,8 +219,8 @@
       effort="1.0"
       velocity="0.5"/>
-    <mimic
+    <!-- <mimic
       joint="left_thumb_proximal_pitch_joint"
       multiplier="1.334"
-      offset="0"/>
+      offset="0"/> -->
   </joint>
   <link
@@ -257,8 +257,8 @@
       effort="1.0"
       velocity="0.5"/>
-    <mimic
+    <!-- <mimic
       joint="left_thumb_proximal_pitch_joint"
       multiplier="0.667"
-      offset="0"/>
+      offset="0"/> -->
   </joint>
   <link
@@ -332,8 +332,8 @@
       effort="1.0"
       velocity="0.5"/>
-    <mimic
+    <!-- <mimic
       joint="left_index_proximal_joint"
       multiplier="1.06399"
-      offset="-0.04545"/>
+      offset="-0.04545"/> -->
   </joint>
   <link
@@ -407,8 +407,8 @@
       effort="1.0"
       velocity="0.5"/>
-    <mimic
+    <!-- <mimic
       joint="left_middle_proximal_joint"
       multiplier="1.06399"
-      offset="-0.04545"/>
+      offset="-0.04545"/> -->
   </joint>
   <link
@@ -483,8 +483,8 @@
       effort="1.0"
       velocity="0.5"/>
-    <mimic
+    <!-- <mimic
       joint="left_ring_proximal_joint"
       multiplier="1.06399"
-      offset="-0.04545"/>
+      offset="-0.04545"/> -->
   </joint>
   <link
@@ -558,8 +558,8 @@
       effort="1.0"
       velocity="0.5"/>
-    <mimic
+    <!-- <mimic
       joint="left_pinky_proximal_joint"
       multiplier="1.06399"
-      offset="-0.04545"/>
+      offset="-0.04545"/> -->
   </joint>
   <link

File: ros2_rm_robot/dual_rm_description/dual_rm_65b_description/urdf/right_hand.urdf.xacro (robot description, xacro)
@@ -219,8 +219,8 @@
       effort="1.0"
       velocity="0.5"/>
-    <mimic
+    <!-- <mimic
       joint="right_thumb_proximal_pitch_joint"
       multiplier="1.334"
-      offset="0"/>
+      offset="0"/> -->
   </joint>
   <link
@@ -257,8 +257,8 @@
       effort="1.0"
       velocity="0.5"/>
-    <mimic
+    <!-- <mimic
       joint="right_thumb_proximal_pitch_joint"
       multiplier="0.667"
-      offset="0"/>
+      offset="0"/> -->
   </joint>
   <link
@@ -333,8 +333,8 @@
       effort="1.0"
       velocity="0.5"/>
-    <mimic
+    <!-- <mimic
       joint="right_index_proximal_joint"
       multiplier="1.06399"
-      offset="-0.04545"/>
+      offset="-0.04545"/> -->
   </joint>
   <link
@@ -409,8 +409,8 @@
       effort="1.0"
       velocity="0.5"/>
-    <mimic
+    <!-- <mimic
       joint="right_middle_proximal_joint"
       multiplier="1.06399"
-      offset="-0.04545"/>
+      offset="-0.04545"/> -->
   </joint>
   <link
@@ -483,8 +483,8 @@
       effort="1.0"
       velocity="0.5"/>
-    <mimic
+    <!-- <mimic
       joint="right_ring_proximal_joint"
       multiplier="1.06399"
-      offset="-0.04545"/>
+      offset="-0.04545"/> -->
   </joint>
   <link
@@ -559,8 +559,8 @@
       effort="1.0"
       velocity="0.5"/>
-    <mimic
+    <!-- <mimic
       joint="right_pinky_proximal_joint"
       multiplier="1.06399"
-      offset="-0.04545"/>
+      offset="-0.04545"/> -->
   </joint>
   <link

File: ros2_rm_robot/dual_rm_moveit_config/dual_rm_65b_moveit_config/config/dual_rm_65b_description.ros2_control.xacro (robot description, xacro)
@@ -64,5 +64,5 @@
                 <state_interface name="velocity"/>
             </joint>
-            <!-- <joint name="left_thumb_intermediate_joint">
+            <joint name="left_thumb_intermediate_joint">
                 <command_interface name="position"/>
                 <state_interface name="position">
@@ -77,5 +77,5 @@
                 </state_interface>
                 <state_interface name="velocity"/>
-            </joint> -->
+            </joint>
             <joint name="left_index_proximal_joint">
                 <command_interface name="position"/>
@@ -85,5 +85,5 @@
                 <state_interface name="velocity"/>
             </joint>
-            <!-- <joint name="left_index_intermediate_joint">
+            <joint name="left_index_intermediate_joint">
                 <command_interface name="position"/>
                 <state_interface name="position">
@@ -91,5 +91,5 @@
                 </state_interface>
                 <state_interface name="velocity"/>
-            </joint> -->
+            </joint>
             <joint name="left_middle_proximal_joint">
                 <command_interface name="position"/>
@@ -99,5 +99,5 @@
                 <state_interface name="velocity"/>
             </joint>
-            <!-- <joint name="left_middle_intermediate_joint">
+            <joint name="left_middle_intermediate_joint">
                 <command_interface name="position"/>
                 <state_interface name="position">
@@ -105,5 +105,5 @@
                 </state_interface>
                 <state_interface name="velocity"/>
-            </joint> -->
+            </joint>
             <joint name="left_ring_proximal_joint">
                 <command_interface name="position"/>
@@ -113,5 +113,5 @@
                 <state_interface name="velocity"/>
             </joint>
-            <!-- <joint name="left_ring_intermediate_joint">
+            <joint name="left_ring_intermediate_joint">
                 <command_interface name="position"/>
                 <state_interface name="position">
@@ -119,5 +119,5 @@
                 </state_interface>
                 <state_interface name="velocity"/>
-            </joint> -->
+            </joint>
             <joint name="left_pinky_proximal_joint">
                 <command_interface name="position"/>
@@ -127,5 +127,5 @@
                 <state_interface name="velocity"/>
             </joint>
-            <!-- <joint name="left_pinky_intermediate_joint">
+            <joint name="left_pinky_intermediate_joint">
                 <command_interface name="position"/>
                 <state_interface name="position">
@@ -133,5 +133,5 @@
                 </state_interface>
                 <state_interface name="velocity"/>
-            </joint> -->
+            </joint>
             <joint name="r_joint1">
                 <command_interface name="position"/>
@@ -190,5 +190,5 @@
                 <state_interface name="velocity"/>
             </joint>
-            <!-- <joint name="right_thumb_intermediate_joint">
+            <joint name="right_thumb_intermediate_joint">
                 <command_interface name="position"/>
                 <state_interface name="position">
@@ -203,5 +203,5 @@
                 </state_interface>
                 <state_interface name="velocity"/>
-            </joint> -->
+            </joint>
             <joint name="right_index_proximal_joint">
                 <command_interface name="position"/>
@@ -211,5 +211,5 @@
                 <state_interface name="velocity"/>
             </joint>
-            <!-- <joint name="right_index_intermediate_joint">
+            <joint name="right_index_intermediate_joint">
                 <command_interface name="position"/>
                 <state_interface name="position">
@@ -217,5 +217,5 @@
                 </state_interface>
                 <state_interface name="velocity"/>
-            </joint> -->
+            </joint>
             <joint name="right_middle_proximal_joint">
                 <command_interface name="position"/>
@@ -225,5 +225,5 @@
                 <state_interface name="velocity"/>
             </joint>
-            <!-- <joint name="right_middle_intermediate_joint">
+            <joint name="right_middle_intermediate_joint">
                 <command_interface name="position"/>
                 <state_interface name="position">
@@ -231,5 +231,5 @@
                 </state_interface>
                 <state_interface name="velocity"/>
-            </joint> -->
+            </joint>
             <joint name="right_ring_proximal_joint">
                 <command_interface name="position"/>
@@ -239,5 +239,5 @@
                 <state_interface name="velocity"/>
             </joint>
-            <!-- <joint name="right_ring_intermediate_joint">
+            <joint name="right_ring_intermediate_joint">
                 <command_interface name="position"/>
                 <state_interface name="position">
@@ -245,5 +245,5 @@
                 </state_interface>
                 <state_interface name="velocity"/>
-            </joint> -->
+            </joint>
             <joint name="right_pinky_proximal_joint">
                 <command_interface name="position"/>
@@ -253,5 +253,5 @@
                 <state_interface name="velocity"/>
             </joint>
-            <!-- <joint name="right_pinky_intermediate_joint">
+            <joint name="right_pinky_intermediate_joint">
                 <command_interface name="position"/>
                 <state_interface name="position">
@@ -259,5 +259,5 @@
                 </state_interface>
                 <state_interface name="velocity"/>
-            </joint> -->
+            </joint>
             <joint name="platform_joint">
                 <command_interface name="position"/>

File: ros2_rm_robot/dual_rm_simulation/dual_rm_65b_gazebo/urdf/depth_camera_65b_gazebo.xacro (robot description, xacro)
@@ -40,4 +40,5 @@
                     <width>1280</width>
                     <height>720</height>
+                    <format>L16</format>
                 </image>
                 <clip>
@@ -51,8 +52,10 @@
                     <remapping>depth/image_raw:=depth/image_rect_raw</remapping>
                     <remapping>depth/camera_info:=depth/camera_info</remapping>
-                    <remapping>points:=depth/color/points</remapping>
+                    <remapping>points:=depth/points</remapping>
                 </ros>
                 <camera_name>depth</camera_name>
                 <frame_name>camera_depth_optical_frame</frame_name>
+                <depth_camera>true</depth_camera>
+                <hack_baseline>0.07</hack_baseline>
                 <min_depth>0.3</min_depth>
                 <max_depth>10.0</max_depth>

File: ros2_rm_robot/dual_rm_simulation/dual_rm_65b_gazebo/urdf/dual_rm_65b_sim.ros2_control.xacro (robot description, xacro)
@@ -61,4 +61,18 @@
             <state_interface name="velocity"/>
         </joint>
+        <joint name="right_thumb_intermediate_joint">
+            <command_interface name="position"/>
+            <state_interface name="position">
+                <param name="initial_value">0</param>
+            </state_interface>
+            <state_interface name="velocity"/>
+        </joint>
+        <joint name="right_thumb_distal_joint">
+            <command_interface name="position"/>
+            <state_interface name="position">
+                <param name="initial_value">0</param>
+            </state_interface>
+            <state_interface name="velocity"/>
+        </joint>
         <joint name="right_index_proximal_joint">
             <command_interface name="position"/>
@@ -68,4 +82,11 @@
             <state_interface name="velocity"/>
         </joint>
+        <joint name="right_index_intermediate_joint">
+            <command_interface name="position"/>
+            <state_interface name="position">
+                <param name="initial_value">0</param>
+            </state_interface>
+            <state_interface name="velocity"/>
+        </joint>
         <joint name="right_middle_proximal_joint">
             <command_interface name="position"/>
@@ -75,4 +96,11 @@
             <state_interface name="velocity"/>
         </joint>
+        <joint name="right_middle_intermediate_joint">
+            <command_interface name="position"/>
+            <state_interface name="position">
+                <param name="initial_value">0</param>
+            </state_interface>
+            <state_interface name="velocity"/>
+        </joint>
         <joint name="right_ring_proximal_joint">
             <command_interface name="position"/>
@@ -82,4 +110,11 @@
             <state_interface name="velocity"/>
         </joint>
+        <joint name="right_ring_intermediate_joint">
+            <command_interface name="position"/>
+            <state_interface name="position">
+                <param name="initial_value">0</param>
+            </state_interface>
+            <state_interface name="velocity"/>
+        </joint>
         <joint name="right_pinky_proximal_joint">
             <command_interface name="position"/>
@@ -89,4 +124,11 @@
             <state_interface name="velocity"/>
         </joint>
+        <joint name="right_pinky_intermediate_joint">
+            <command_interface name="position"/>
+            <state_interface name="position">
+                <param name="initial_value">0</param>
+            </state_interface>
+            <state_interface name="velocity"/>
+        </joint>
         <joint name="l_joint1">
             <command_interface name="position"/>
@@ -145,4 +187,18 @@
             <state_interface name="velocity"/>
         </joint>
+        <joint name="left_thumb_intermediate_joint">
+            <command_interface name="position"/>
+            <state_interface name="position">
+                <param name="initial_value">0</param>
+            </state_interface>
+            <state_interface name="velocity"/>
+        </joint>
+        <joint name="left_thumb_distal_joint">
+            <command_interface name="position"/>
+            <state_interface name="position">
+                <param name="initial_value">0</param>
+            </state_interface>
+            <state_interface name="velocity"/>
+        </joint>
         <joint name="left_index_proximal_joint">
             <command_interface name="position"/>
@@ -152,4 +208,11 @@
             <state_interface name="velocity"/>
         </joint>
+        <joint name="left_index_intermediate_joint">
+            <command_interface name="position"/>
+            <state_interface name="position">
+                <param name="initial_value">0</param>
+            </state_interface>
+            <state_interface name="velocity"/>
+        </joint>
         <joint name="left_middle_proximal_joint">
             <command_interface name="position"/>
@@ -159,4 +222,11 @@
             <state_interface name="velocity"/>
         </joint>
+        <joint name="left_middle_intermediate_joint">
+            <command_interface name="position"/>
+            <state_interface name="position">
+                <param name="initial_value">0</param>
+            </state_interface>
+            <state_interface name="velocity"/>
+        </joint>
         <joint name="left_ring_proximal_joint">
             <command_interface name="position"/>
@@ -166,5 +236,19 @@
             <state_interface name="velocity"/>
         </joint>
+        <joint name="left_ring_intermediate_joint">
+            <command_interface name="position"/>
+            <state_interface name="position">
+                <param name="initial_value">0</param>
+            </state_interface>
+            <state_interface name="velocity"/>
+        </joint>
         <joint name="left_pinky_proximal_joint">
+            <command_interface name="position"/>
+            <state_interface name="position">
+                <param name="initial_value">0</param>
+            </state_interface>
+            <state_interface name="velocity"/>
+        </joint>
+        <joint name="left_pinky_intermediate_joint">
             <command_interface name="position"/>
             <state_interface name="position">
