Commit message: hand integrated with moveit for 65b arm

File: ros2_rm_robot/dual_rm_moveit_config/dual_rm_65b_moveit_config/config/dual_rm_65b_description.ros2_control.xacro (robot description, xacro)
@@ -50,4 +50,88 @@
                 <state_interface name="velocity"/>
             </joint>
+            <joint name="left_thumb_proximal_yaw_joint">
+                <command_interface name="position"/>
+                <state_interface name="position">
+                    <param name="initial_value">${initial_positions['left_thumb_proximal_yaw_joint']}</param>
+                </state_interface>
+                <state_interface name="velocity"/>
+            </joint>
+            <joint name="left_thumb_proximal_pitch_joint">
+                <command_interface name="position"/>
+                <state_interface name="position">
+                    <param name="initial_value">${initial_positions['left_thumb_proximal_pitch_joint']}</param>
+                </state_interface>
+                <state_interface name="velocity"/>
+            </joint>
+            <joint name="left_thumb_intermediate_joint">
+                <command_interface name="position"/>
+                <state_interface name="position">
+                    <param name="initial_value">${initial_positions['left_thumb_intermediate_joint']}</param>
+                </state_interface>
+                <state_interface name="velocity"/>
+            </joint>
+            <joint name="left_thumb_distal_joint">
+                <command_interface name="position"/>
+                <state_interface name="position">
+                    <param name="initial_value">${initial_positions['left_thumb_distal_joint']}</param>
+                </state_interface>
+                <state_interface name="velocity"/>
+            </joint>
+            <joint name="left_index_proximal_joint">
+                <command_interface name="position"/>
+                <state_interface name="position">
+                    <param name="initial_value">${initial_positions['left_index_proximal_joint']}</param>
+                </state_interface>
+                <state_interface name="velocity"/>
+            </joint>
+            <joint name="left_index_intermediate_joint">
+                <command_interface name="position"/>
+                <state_interface name="position">
+                    <param name="initial_value">${initial_positions['left_index_intermediate_joint']}</param>
+                </state_interface>
+                <state_interface name="velocity"/>
+            </joint>
+            <joint name="left_middle_proximal_joint">
+                <command_interface name="position"/>
+                <state_interface name="position">
+                    <param name="initial_value">${initial_positions['left_middle_proximal_joint']}</param>
+                </state_interface>
+                <state_interface name="velocity"/>
+            </joint>
+            <joint name="left_middle_intermediate_joint">
+                <command_interface name="position"/>
+                <state_interface name="position">
+                    <param name="initial_value">${initial_positions['left_middle_intermediate_joint']}</param>
+                </state_interface>
+                <state_interface name="velocity"/>
+            </joint>
+            <joint name="left_ring_proximal_joint">
+                <command_interface name="position"/>
+                <state_interface name="position">
+                    <param name="initial_value">${initial_positions['left_ring_proximal_joint']}</param>
+                </state_interface>
+                <state_interface name="velocity"/>
+            </joint>
+            <joint name="left_ring_intermediate_joint">
+                <command_interface name="position"/>
+                <state_interface name="position">
+                    <param name="initial_value">${initial_positions['left_ring_intermediate_joint']}</param>
+                </state_interface>
+                <state_interface name="velocity"/>
+            </joint>
+            <joint name="left_pinky_proximal_joint">
+                <command_interface name="position"/>
+                <state_interface name="position">
+                    <param name="initial_value">${initial_positions['left_pinky_proximal_joint']}</param>
+                </state_interface>
+                <state_interface name="velocity"/>
+            </joint>
+            <joint name="left_pinky_intermediate_joint">
+                <command_interface name="position"/>
+                <state_interface name="position">
+                    <param name="initial_value">${initial_positions['left_pinky_intermediate_joint']}</param>
+                </state_interface>
+                <state_interface name="velocity"/>
+            </joint>
             <joint name="r_joint1">
                 <command_interface name="position"/>
@@ -89,4 +173,88 @@
                 <state_interface name="position">
                   <param name="initial_value">${initial_positions['r_joint6']}</param>
+                </state_interface>
+                <state_interface name="velocity"/>
+            </joint>
+            <joint name="right_thumb_proximal_yaw_joint">
+                <command_interface name="position"/>
+                <state_interface name="position">
+                    <param name="initial_value">${initial_positions['right_thumb_proximal_yaw_joint']}</param>
+                </state_interface>
+                <state_interface name="velocity"/>
+            </joint>
+            <joint name="right_thumb_proximal_pitch_joint">
+                <command_interface name="position"/>
+                <state_interface name="position">
+                    <param name="initial_value">${initial_positions['right_thumb_proximal_pitch_joint']}</param>
+                </state_interface>
+                <state_interface name="velocity"/>
+            </joint>
+            <joint name="right_thumb_intermediate_joint">
+                <command_interface name="position"/>
+                <state_interface name="position">
+                    <param name="initial_value">${initial_positions['right_thumb_intermediate_joint']}</param>
+                </state_interface>
+                <state_interface name="velocity"/>
+            </joint>
+            <joint name="right_thumb_distal_joint">
+                <command_interface name="position"/>
+                <state_interface name="position">
+                    <param name="initial_value">${initial_positions['right_thumb_distal_joint']}</param>
+                </state_interface>
+                <state_interface name="velocity"/>
+            </joint>
+            <joint name="right_index_proximal_joint">
+                <command_interface name="position"/>
+                <state_interface name="position">
+                    <param name="initial_value">${initial_positions['right_index_proximal_joint']}</param>
+                </state_interface>
+                <state_interface name="velocity"/>
+            </joint>
+            <joint name="right_index_intermediate_joint">
+                <command_interface name="position"/>
+                <state_interface name="position">
+                    <param name="initial_value">${initial_positions['right_index_intermediate_joint']}</param>
+                </state_interface>
+                <state_interface name="velocity"/>
+            </joint>
+            <joint name="right_middle_proximal_joint">
+                <command_interface name="position"/>
+                <state_interface name="position">
+                    <param name="initial_value">${initial_positions['right_middle_proximal_joint']}</param>
+                </state_interface>
+                <state_interface name="velocity"/>
+            </joint>
+            <joint name="right_middle_intermediate_joint">
+                <command_interface name="position"/>
+                <state_interface name="position">
+                    <param name="initial_value">${initial_positions['right_middle_intermediate_joint']}</param>
+                </state_interface>
+                <state_interface name="velocity"/>
+            </joint>
+            <joint name="right_ring_proximal_joint">
+                <command_interface name="position"/>
+                <state_interface name="position">
+                    <param name="initial_value">${initial_positions['right_ring_proximal_joint']}</param>
+                </state_interface>
+                <state_interface name="velocity"/>
+            </joint>
+            <joint name="right_ring_intermediate_joint">
+                <command_interface name="position"/>
+                <state_interface name="position">
+                    <param name="initial_value">${initial_positions['right_ring_intermediate_joint']}</param>
+                </state_interface>
+                <state_interface name="velocity"/>
+            </joint>
+            <joint name="right_pinky_proximal_joint">
+                <command_interface name="position"/>
+                <state_interface name="position">
+                    <param name="initial_value">${initial_positions['right_pinky_proximal_joint']}</param>
+                </state_interface>
+                <state_interface name="velocity"/>
+            </joint>
+            <joint name="right_pinky_intermediate_joint">
+                <command_interface name="position"/>
+                <state_interface name="position">
+                    <param name="initial_value">${initial_positions['right_pinky_intermediate_joint']}</param>
                 </state_interface>
                 <state_interface name="velocity"/>

File: ros2_rm_robot/dual_rm_simulation/dual_rm_65b_gazebo/urdf/dual_rm_65b_sim.ros2_control.xacro (robot description, xacro)
@@ -188,11 +188,4 @@
         </joint>
         <joint name="left_thumb_intermediate_joint">
-            <command_interface name="position"/>
-            <state_interface name="position">
-                <param name="initial_value">0</param>
-            </state_interface>
-            <state_interface name="velocity"/>
-        </joint>
-        <joint name="left_thumb_proximal_yaw_joint">
             <command_interface name="position"/>
             <state_interface name="position">

Commit message: hand_moveit worked

File: ros2_rm_robot/dual_rm_moveit_config/dual_rm_65b_moveit_config/config/dual_rm_65b_description.ros2_control.xacro (robot description, xacro)
@@ -64,5 +64,5 @@
                 <state_interface name="velocity"/>
             </joint>
-            <joint name="left_thumb_intermediate_joint">
+            <!-- <joint name="left_thumb_intermediate_joint">
                 <command_interface name="position"/>
                 <state_interface name="position">
@@ -77,5 +77,5 @@
                 </state_interface>
                 <state_interface name="velocity"/>
-            </joint>
+            </joint> -->
             <joint name="left_index_proximal_joint">
                 <command_interface name="position"/>
@@ -85,5 +85,5 @@
                 <state_interface name="velocity"/>
             </joint>
-            <joint name="left_index_intermediate_joint">
+            <!-- <joint name="left_index_intermediate_joint">
                 <command_interface name="position"/>
                 <state_interface name="position">
@@ -91,5 +91,5 @@
                 </state_interface>
                 <state_interface name="velocity"/>
-            </joint>
+            </joint> -->
             <joint name="left_middle_proximal_joint">
                 <command_interface name="position"/>
@@ -99,5 +99,5 @@
                 <state_interface name="velocity"/>
             </joint>
-            <joint name="left_middle_intermediate_joint">
+            <!-- <joint name="left_middle_intermediate_joint">
                 <command_interface name="position"/>
                 <state_interface name="position">
@@ -105,5 +105,5 @@
                 </state_interface>
                 <state_interface name="velocity"/>
-            </joint>
+            </joint> -->
             <joint name="left_ring_proximal_joint">
                 <command_interface name="position"/>
@@ -113,5 +113,5 @@
                 <state_interface name="velocity"/>
             </joint>
-            <joint name="left_ring_intermediate_joint">
+            <!-- <joint name="left_ring_intermediate_joint">
                 <command_interface name="position"/>
                 <state_interface name="position">
@@ -119,5 +119,5 @@
                 </state_interface>
                 <state_interface name="velocity"/>
-            </joint>
+            </joint> -->
             <joint name="left_pinky_proximal_joint">
                 <command_interface name="position"/>
@@ -127,5 +127,5 @@
                 <state_interface name="velocity"/>
             </joint>
-            <joint name="left_pinky_intermediate_joint">
+            <!-- <joint name="left_pinky_intermediate_joint">
                 <command_interface name="position"/>
                 <state_interface name="position">
@@ -133,5 +133,5 @@
                 </state_interface>
                 <state_interface name="velocity"/>
-            </joint>
+            </joint> -->
             <joint name="r_joint1">
                 <command_interface name="position"/>
@@ -190,5 +190,5 @@
                 <state_interface name="velocity"/>
             </joint>
-            <joint name="right_thumb_intermediate_joint">
+            <!-- <joint name="right_thumb_intermediate_joint">
                 <command_interface name="position"/>
                 <state_interface name="position">
@@ -203,5 +203,5 @@
                 </state_interface>
                 <state_interface name="velocity"/>
-            </joint>
+            </joint> -->
             <joint name="right_index_proximal_joint">
                 <command_interface name="position"/>
@@ -211,5 +211,5 @@
                 <state_interface name="velocity"/>
             </joint>
-            <joint name="right_index_intermediate_joint">
+            <!-- <joint name="right_index_intermediate_joint">
                 <command_interface name="position"/>
                 <state_interface name="position">
@@ -217,5 +217,5 @@
                 </state_interface>
                 <state_interface name="velocity"/>
-            </joint>
+            </joint> -->
             <joint name="right_middle_proximal_joint">
                 <command_interface name="position"/>
@@ -225,5 +225,5 @@
                 <state_interface name="velocity"/>
             </joint>
-            <joint name="right_middle_intermediate_joint">
+            <!-- <joint name="right_middle_intermediate_joint">
                 <command_interface name="position"/>
                 <state_interface name="position">
@@ -231,5 +231,5 @@
                 </state_interface>
                 <state_interface name="velocity"/>
-            </joint>
+            </joint> -->
             <joint name="right_ring_proximal_joint">
                 <command_interface name="position"/>
@@ -239,5 +239,5 @@
                 <state_interface name="velocity"/>
             </joint>
-            <joint name="right_ring_intermediate_joint">
+            <!-- <joint name="right_ring_intermediate_joint">
                 <command_interface name="position"/>
                 <state_interface name="position">
@@ -245,5 +245,5 @@
                 </state_interface>
                 <state_interface name="velocity"/>
-            </joint>
+            </joint> -->
             <joint name="right_pinky_proximal_joint">
                 <command_interface name="position"/>
@@ -253,5 +253,5 @@
                 <state_interface name="velocity"/>
             </joint>
-            <joint name="right_pinky_intermediate_joint">
+            <!-- <joint name="right_pinky_intermediate_joint">
                 <command_interface name="position"/>
                 <state_interface name="position">
@@ -259,5 +259,5 @@
                 </state_interface>
                 <state_interface name="velocity"/>
-            </joint>
+            </joint> -->
             <joint name="platform_joint">
                 <command_interface name="position"/>

File: ros2_rm_robot/dual_rm_simulation/dual_rm_65b_gazebo/urdf/dual_rm_65b_gazebo.urdf.xacro (robot description, xacro)
@@ -1,7 +1,7 @@
 <?xml version="1.0"?>
 <robot xmlns:xacro="http://www.ros.org/wiki/xacro" name="dual_rm_65b_gazebo">
-    <link name="base_footprint"/>
-    <joint name="base_footprint_to_base_link" type="fixed">
-        <parent link="base_footprint"/>
+    <link name="world"/>
+    <joint name="world_to_base_link" type="fixed">
+        <parent link="world"/>
         <child link="base_link_underpan"/>
         <origin xyz="0 0 0" rpy="0 0 0"/>

File: ros2_rm_robot/dual_rm_simulation/dual_rm_65b_gazebo/urdf/dual_rm_65b_sim.ros2_control.xacro (robot description, xacro)
@@ -61,18 +61,4 @@
             <state_interface name="velocity"/>
         </joint>
-        <joint name="right_thumb_intermediate_joint">
-            <command_interface name="position"/>
-            <state_interface name="position">
-                <param name="initial_value">0</param>
-            </state_interface>
-            <state_interface name="velocity"/>
-        </joint>
-        <joint name="right_thumb_distal_joint">
-            <command_interface name="position"/>
-            <state_interface name="position">
-                <param name="initial_value">0</param>
-            </state_interface>
-            <state_interface name="velocity"/>
-        </joint>
         <joint name="right_index_proximal_joint">
             <command_interface name="position"/>
@@ -82,11 +68,4 @@
             <state_interface name="velocity"/>
         </joint>
-        <joint name="right_index_intermediate_joint">
-            <command_interface name="position"/>
-            <state_interface name="position">
-                <param name="initial_value">0</param>
-            </state_interface>
-            <state_interface name="velocity"/>
-        </joint>
         <joint name="right_middle_proximal_joint">
             <command_interface name="position"/>
@@ -96,11 +75,4 @@
             <state_interface name="velocity"/>
         </joint>
-        <joint name="right_middle_intermediate_joint">
-            <command_interface name="position"/>
-            <state_interface name="position">
-                <param name="initial_value">0</param>
-            </state_interface>
-            <state_interface name="velocity"/>
-        </joint>
         <joint name="right_ring_proximal_joint">
             <command_interface name="position"/>
@@ -110,11 +82,4 @@
             <state_interface name="velocity"/>
         </joint>
-        <joint name="right_ring_intermediate_joint">
-            <command_interface name="position"/>
-            <state_interface name="position">
-                <param name="initial_value">0</param>
-            </state_interface>
-            <state_interface name="velocity"/>
-        </joint>
         <joint name="right_pinky_proximal_joint">
             <command_interface name="position"/>
@@ -124,11 +89,4 @@
             <state_interface name="velocity"/>
         </joint>
-        <joint name="right_pinky_intermediate_joint">
-            <command_interface name="position"/>
-            <state_interface name="position">
-                <param name="initial_value">0</param>
-            </state_interface>
-            <state_interface name="velocity"/>
-        </joint>
         <joint name="l_joint1">
             <command_interface name="position"/>
@@ -187,18 +145,4 @@
             <state_interface name="velocity"/>
         </joint>
-        <joint name="left_thumb_intermediate_joint">
-            <command_interface name="position"/>
-            <state_interface name="position">
-                <param name="initial_value">0</param>
-            </state_interface>
-            <state_interface name="velocity"/>
-        </joint>
-        <joint name="left_thumb_distal_joint">
-            <command_interface name="position"/>
-            <state_interface name="position">
-                <param name="initial_value">0</param>
-            </state_interface>
-            <state_interface name="velocity"/>
-        </joint>
         <joint name="left_index_proximal_joint">
             <command_interface name="position"/>
@@ -208,11 +152,4 @@
             <state_interface name="velocity"/>
         </joint>
-        <joint name="left_index_intermediate_joint">
-            <command_interface name="position"/>
-            <state_interface name="position">
-                <param name="initial_value">0</param>
-            </state_interface>
-            <state_interface name="velocity"/>
-        </joint>
         <joint name="left_middle_proximal_joint">
             <command_interface name="position"/>
@@ -222,11 +159,4 @@
             <state_interface name="velocity"/>
         </joint>
-        <joint name="left_middle_intermediate_joint">
-            <command_interface name="position"/>
-            <state_interface name="position">
-                <param name="initial_value">0</param>
-            </state_interface>
-            <state_interface name="velocity"/>
-        </joint>
         <joint name="left_ring_proximal_joint">
             <command_interface name="position"/>
@@ -236,19 +166,5 @@
             <state_interface name="velocity"/>
         </joint>
-        <joint name="left_ring_intermediate_joint">
-            <command_interface name="position"/>
-            <state_interface name="position">
-                <param name="initial_value">0</param>
-            </state_interface>
-            <state_interface name="velocity"/>
-        </joint>
         <joint name="left_pinky_proximal_joint">
-            <command_interface name="position"/>
-            <state_interface name="position">
-                <param name="initial_value">0</param>
-            </state_interface>
-            <state_interface name="velocity"/>
-        </joint>
-        <joint name="left_pinky_intermediate_joint">
             <command_interface name="position"/>
             <state_interface name="position">

File: ros2_rm_robot/dual_rm_simulation/dual_rm_75b_gazebo/urdf/dual_rm_75b_gazebo.urdf.xacro (robot description, xacro)
@@ -1,7 +1,7 @@
 <?xml version="1.0"?>
 <robot xmlns:xacro="http://www.ros.org/wiki/xacro" name="dual_rm_75b_gazebo">
-    <link name="base_footprint"/>
-    <joint name="base_footprint_to_base_link" type="fixed">
-        <parent link="base_footprint"/>
+    <link name="world"/>
+    <joint name="world_to_base_link" type="fixed">
+        <parent link="world"/>
         <child link="base_link_underpan"/>
         <origin xyz="0 0 0" rpy="0 0 0"/>
