Commit message: minimized code duplication
Signed-off-by: Nitin <nitinmaurya2606@gmail.com>

File: ros2_rm_robot/dual_rm_moveit_config/dual_rm_65b_moveit_config/config/dual_rm_65b_description.urdf.xacro (robot description, xacro)
@@ -2,6 +2,7 @@
 <robot xmlns:xacro="http://www.ros.org/wiki/xacro" name="dual_rm_65b_description">
     <xacro:arg name="initial_positions_file" default="initial_positions.yaml" />
-    <!-- Import dual_rm_65b_description urdf file -->
-    <xacro:include filename="$(find dual_rm_65b_description)/urdf/dual_rm_65b_description.urdf.xacro" />
+    <!-- Import robot description (unified package, 65b variant) -->
+    <xacro:arg name="arm_model" default="65b"/>
+    <xacro:include filename="$(find dual_rm_description)/urdf/r2d3_description.urdf.xacro" />
     <!-- Import control_xacro -->
     <xacro:include filename="dual_rm_65b_description.ros2_control.xacro" />

File: ros2_rm_robot/dual_rm_moveit_config/dual_rm_75b_moveit_config/config/dual_rm_75b_description.urdf.xacro (robot description, xacro)
@@ -2,6 +2,7 @@
 <robot xmlns:xacro="http://www.ros.org/wiki/xacro" name="dual_rm_75b_description">
     <xacro:arg name="initial_positions_file" default="initial_positions.yaml" />
-    <!-- Import dual_rm_75b_description urdf file -->
-    <xacro:include filename="$(find dual_rm_75b_description)/urdf/dual_rm_75b_description.urdf.xacro" />
+    <!-- Import robot description (unified package, 75b variant) -->
+    <xacro:arg name="arm_model" default="75b"/>
+    <xacro:include filename="$(find dual_rm_description)/urdf/r2d3_description.urdf.xacro" />
     <!-- Import control_xacro -->
     <xacro:include filename="dual_rm_75b_description.ros2_control.xacro" />

File: ros2_rm_robot/dual_rm_simulation/urdf/gazebo/sim_gazebo.urdf.xacro (robot description, xacro)
@@ -1,8 +1,4 @@
 <?xml version="1.0"?>
 <!--
-  Gazebo Sim physics properties for R2D3 navigation simulation.
-  Sets self_collide, friction (mu1/mu2), and gravity overrides for every
-  link that needs them.  Parameterised by arm_dof so the same file works
-  for both the 65b (6-DOF arms) and 75b (7-DOF arms) variants.
   Usage:
     <xacro:include filename=".../gazebo/sim_gazebo.urdf.xacro"/>
@@ -11,5 +7,4 @@
 -->
 <robot xmlns:xacro="http://www.ros.org/wiki/xacro">
-    <!-- ── Helper: mark a link as no-gravity, no-self-collide ── -->
     <xacro:macro name="_gz_no_gravity" params="link_name">
         <gazebo reference="${link_name}">
@@ -19,5 +14,5 @@
     </xacro:macro>
     <!-- ── Helper: caster wheel friction ─────────────────────── -->
-    <xacro:macro name="_gz_caster" params="link_name">
+    <xacro:macro name="_gz_caster_bracket" params="link_name">
         <gazebo reference="${link_name}">
             <self_collide>false</self_collide>
@@ -26,7 +21,12 @@
         </gazebo>
     </xacro:macro>
-    <!-- ============================================================
-         Main macro
-         ============================================================ -->
+    <!-- Caster wheels (sphere collision): moderate friction for stability -->
+    <xacro:macro name="_gz_caster_wheel" params="link_name">
+        <gazebo reference="${link_name}">
+            <self_collide>false</self_collide>
+            <mu1>0.3</mu1>
+            <mu2>0.3</mu2>
+        </gazebo>
+    </xacro:macro>
     <xacro:macro name="sim_gazebo_properties" params="arm_dof">
         <!-- ── Robot-level ───────────────────────────────────── -->
@@ -46,24 +46,25 @@
             <gravity>false</gravity>
         </gazebo>
-        <!-- ── Drive wheels (high friction) ──────────────────── -->
+        <!-- ── Drive wheels (high friction for traction) ─────── -->
         <gazebo reference="link_right_wheel">
             <self_collide>false</self_collide>
-            <mu1>1.0</mu1>
-            <mu2>1.0</mu2>
+            <mu1>1.5</mu1>
+            <mu2>1.5</mu2>
         </gazebo>
         <gazebo reference="link_left_wheel">
             <self_collide>false</self_collide>
-            <mu1>1.0</mu1>
-            <mu2>1.0</mu2>
+            <mu1>1.5</mu1>
+            <mu2>1.5</mu2>
         </gazebo>
-        <!-- ── Caster / swivel wheels (low friction) ─────────── -->
-        <xacro:_gz_caster link_name="link_swivel_wheel_1_1"/>
-        <xacro:_gz_caster link_name="link_swivel_wheel_1_2"/>
-        <xacro:_gz_caster link_name="link_swivel_wheel_2_1"/>
-        <xacro:_gz_caster link_name="link_swivel_wheel_2_2"/>
-        <xacro:_gz_caster link_name="link_swivel_wheel_3_1"/>
-        <xacro:_gz_caster link_name="link_swivel_wheel_3_2"/>
-        <xacro:_gz_caster link_name="link_swivel_wheel_4_1"/>
-        <xacro:_gz_caster link_name="link_swivel_wheel_4_2"/>
+        <!-- ── Caster brackets (swivel forks, low friction) ──── -->
+        <xacro:_gz_caster_bracket link_name="link_swivel_wheel_1_1"/>
+        <xacro:_gz_caster_bracket link_name="link_swivel_wheel_2_1"/>
+        <xacro:_gz_caster_bracket link_name="link_swivel_wheel_3_1"/>
+        <xacro:_gz_caster_bracket link_name="link_swivel_wheel_4_1"/>
+        <!-- ── Caster wheels (sphere collision, moderate friction) -->
+        <xacro:_gz_caster_wheel link_name="link_swivel_wheel_1_2"/>
+        <xacro:_gz_caster_wheel link_name="link_swivel_wheel_2_2"/>
+        <xacro:_gz_caster_wheel link_name="link_swivel_wheel_3_2"/>
+        <xacro:_gz_caster_wheel link_name="link_swivel_wheel_4_2"/>
         <!-- ── Arm links (no gravity) ────────────────────────── -->
         <!-- Common to both 65b and 75b: links 1-6 -->

File: ros2_rm_robot/dual_rm_simulation/urdf/ros2_control/sim_ros2_control.urdf.xacro (robot description, xacro)
@@ -1,8 +1,4 @@
 <?xml version="1.0"?>
 <!--
-  ros2_control hardware interface + gz_ros2_control plugin for R2D3 sim.
-  Defines command/state interfaces for every actuated and passive joint.
-  Parameterised by arm_dof (6 for 65b, 7 for 75b) and the path to the
-  controller-manager YAML so both robot variants share one file.
   Usage:
     <xacro:include filename=".../ros2_control/sim_ros2_control.urdf.xacro"/>
@@ -21,5 +17,4 @@
         </joint>
     </xacro:macro>
-    <!-- ── Helper: passive (state-only) caster joint ─────────── -->
     <xacro:macro name="_passive_joint" params="joint_name">
         <joint name="${joint_name}">
@@ -30,7 +25,4 @@
         </joint>
     </xacro:macro>
-    <!-- ============================================================
-         Main macro
-         ============================================================ -->
     <xacro:macro name="sim_ros2_control" params="arm_dof controllers_yaml">
         <ros2_control name="GazeboSimSystem" type="system">

File: ros2_rm_robot/dual_rm_simulation/urdf/sensors/imu.urdf.xacro (robot description, xacro)
@@ -2,9 +2,4 @@
 <!--
   IMU sensor macro for R2D3 navigation simulation (Gz Sim / Harmonic).
-  Provides:
-    - imu_link          (inertial only, no visual)
-    - imu_joint         (fixed, attached to parent_link)
-    - Gazebo imu sensor plugin
-    - Gazebo reference  properties (no self-collide, no gravity)
   Usage:
     <xacro:include filename=".../sensors/imu.urdf.xacro"/>

File: ros2_rm_robot/dual_rm_simulation/urdf/sensors/lidar.urdf.xacro (robot description, xacro)
@@ -2,9 +2,4 @@
 <!--
   LiDAR sensor macro for R2D3 navigation simulation (Gz Sim / Harmonic).
-  Provides:
-    - lidar_link         (visual cylinder + collision + inertial)
-    - lidar_joint        (fixed, attached to parent_link)
-    - Gazebo gpu_lidar   sensor plugin (360° scan)
-    - Gazebo reference   properties (no self-collide, no gravity)
   Usage:
     <xacro:include filename=".../sensors/lidar.urdf.xacro"/>
