Commit message: Refactored Description
Signed-off-by: Nitin <nitinmaurya2606@gmail.com>

File: ros2_rm_robot/dual_rm_description/dual_rm_65b_description/urdf/agv/woosh_agv.urdf.xacro (robot description, xacro)
@@ -2,5 +2,5 @@
 <robot name="woosh_agv" xmlns:xacro="http://www.ros.org/wiki/xacro">
   <!-- Define constants -->
-  <xacro:property name="mesh_path" value="file://$(find dual_rm_75b_description)/meshes/" />
+  <xacro:property name="mesh_path" value="file://$(find dual_rm_65b_description)/meshes/" />
   <!-- Macro for visual and collision elements -->
   <xacro:macro name="visual_collision" params="mesh">
@@ -39,4 +39,6 @@
     <xacro:visual_collision mesh="base_link_underpan.STL" />
   </link>
+  <!-- Drive wheels: mesh for visual, CYLINDER for collision (reliable rolling contact in Gz Sim) -->
+  <!-- Wheel geometry: radius=0.08m, width≈0.05m, axis along X -->
   <link
     name="link_right_wheel">
@@ -55,5 +57,20 @@
         izz="0.0018066" />
     </inertial>
-    <xacro:visual_collision mesh="link_right_wheel.STL" />
+    <visual>
+      <origin xyz="0 0 0" rpy="0 0 0" />
+      <geometry>
+        <mesh filename="${mesh_path}link_right_wheel.STL" />
+      </geometry>
+      <material name="">
+        <color rgba="0.79216 0.81961 0.93333 1" />
+      </material>
+    </visual>
+    <collision>
+      <!-- Cylinder along X axis: rotate 90° around Y -->
+      <origin xyz="-0.025 0 0" rpy="0 ${pi/2} 0" />
+      <geometry>
+        <cylinder radius="0.08" length="0.05" />
+      </geometry>
+    </collision>
   </link>
   <link
@@ -73,5 +90,20 @@
         izz="0.0019593" />
     </inertial>
-    <xacro:visual_collision mesh="link_left_wheel.STL" />
+    <visual>
+      <origin xyz="0 0 0" rpy="0 0 0" />
+      <geometry>
+        <mesh filename="${mesh_path}link_left_wheel.STL" />
+      </geometry>
+      <material name="">
+        <color rgba="0.79216 0.81961 0.93333 1" />
+      </material>
+    </visual>
+    <collision>
+      <!-- Cylinder along X axis: rotate 90° around Y -->
+      <origin xyz="0.025 0 0" rpy="0 ${pi/2} 0" />
+      <geometry>
+        <cylinder radius="0.08" length="0.05" />
+      </geometry>
+    </collision>
   </link>
   <link
@@ -165,5 +197,5 @@
     <xacro:visual_collision mesh="link_swivel_wheel_3_1.STL" />
   </link>
-   <link
+  <link
     name="link_swivel_wheel_3_2">
     <inertial>
@@ -246,5 +278,5 @@
       link="link_left_wheel" />
     <axis
-      xyz="-1 0 0" />
+      xyz="1 0 0" />
     <limit
       effort="100"
@@ -303,5 +335,5 @@
       xyz="1 0 0" />
   </joint>
-   <joint
+  <joint
     name="joint_swivel_wheel_3_1"
     type="continuous">

File: ros2_rm_robot/dual_rm_description/dual_rm_65b_description/urdf/dual_rm_65b_description.urdf.xacro (robot description, xacro)
@@ -1,17 +1,32 @@
 <?xml version="1.0"?>
+<!--
+  R2D3 65b Robot Description — main xacro entry point.
+  Assembles the full robot from modular sub-components:
+    agv/            — AGV chassis, drive wheels, caster wheels
+    body/           — Torso, head, camera, platform lift
+    left_arm/       — Left 6-DOF arm + gripper
+    right_arm/      — Right 6-DOF arm + gripper
+    joints/         — Cross-component joints (body↔arms, arms↔hands)
+    materials/      — Named URDF colour definitions
+    transmissions/  — Legacy ROS1 transmission tags (kept for compatibility)
+-->
 <robot name="dual_rm_65b_description" xmlns:xacro="http://ros.org/wiki/xacro">
-  <!-- 引入各个模块的 xacro 文件，分别定义底盘、夹爪、升降平台、机械臂及关节 -->
-  <xacro:include filename="$(find dual_rm_65b_description)/urdf/woosh_agv.urdf.xacro"/>
-  <xacro:include filename="$(find dual_rm_65b_description)/urdf/body_head_platform.urdf.xacro"/>
-  <xacro:include filename="$(find dual_rm_65b_description)/urdf/left_hand.urdf.xacro"/>
-  <xacro:include filename="$(find dual_rm_65b_description)/urdf/right_hand.urdf.xacro"/>
-  <xacro:include filename="$(find dual_rm_65b_description)/urdf/rm65_b_v_left.urdf.xacro"/>
-  <xacro:include filename="$(find dual_rm_65b_description)/urdf/rm65_b_v_right.urdf.xacro"/>
-  <xacro:include filename="$(find dual_rm_65b_description)/urdf/joint.urdf.xacro"/>
-  <!-- 在 Gazebo 仿真环境中添加控制传动配置及 Gazebo 专用插件 -->
-  <xacro:include filename="$(find dual_rm_65b_description)/urdf/rm65_b_v_left_transmission.xacro"/>
-  <xacro:include filename="$(find dual_rm_65b_description)/urdf/rm65_b_v_right_transmission.xacro"/>
-  <xacro:include filename="$(find dual_rm_65b_description)/urdf/body_head_platform_transmission.xacro"/>
-  <!-- Gazebo Classic plugin - not available on Jazzy (Gz Sim Harmonic only) -->
-  <!-- <xacro:include filename="$(find dual_rm_65b_description)/urdf/common_gazebo.xacro"/> -->
+    <!-- ── Materials ─────────────────────────────────────────── -->
+    <xacro:include filename="$(find dual_rm_65b_description)/urdf/materials/colors.urdf.xacro"/>
+    <!-- ── AGV chassis (wheels, casters) ─────────────────────── -->
+    <xacro:include filename="$(find dual_rm_65b_description)/urdf/agv/woosh_agv.urdf.xacro"/>
+    <!-- ── Body, head, camera, platform lift ─────────────────── -->
+    <xacro:include filename="$(find dual_rm_65b_description)/urdf/body/body_head_platform.urdf.xacro"/>
+    <!-- ── Left arm (6-DOF) + gripper ────────────────────────── -->
+    <xacro:include filename="$(find dual_rm_65b_description)/urdf/left_arm/rm65_b_v_left.urdf.xacro"/>
+    <xacro:include filename="$(find dual_rm_65b_description)/urdf/left_arm/left_hand.urdf.xacro"/>
+    <!-- ── Right arm (6-DOF) + gripper ───────────────────────── -->
+    <xacro:include filename="$(find dual_rm_65b_description)/urdf/right_arm/rm65_b_v_right.urdf.xacro"/>
+    <xacro:include filename="$(find dual_rm_65b_description)/urdf/right_arm/right_hand.urdf.xacro"/>
+    <!-- ── Cross-component joints ────────────────────────────── -->
+    <xacro:include filename="$(find dual_rm_65b_description)/urdf/joints/joint.urdf.xacro"/>
+    <!-- ── Transmissions (legacy ROS1, kept for compatibility) ── -->
+    <xacro:include filename="$(find dual_rm_65b_description)/urdf/transmissions/rm65_b_v_left_transmission.xacro"/>
+    <xacro:include filename="$(find dual_rm_65b_description)/urdf/transmissions/rm65_b_v_right_transmission.xacro"/>
+    <xacro:include filename="$(find dual_rm_65b_description)/urdf/transmissions/body_head_platform_transmission.xacro"/>
 </robot>

File: ros2_rm_robot/dual_rm_description/dual_rm_65b_description/urdf/joints/joint.urdf.xacro (robot description, xacro)
@@ -1,5 +1,5 @@
 <?xml version="1.0"?>
 <robot name="joint" xmlns:xacro="http://www.ros.org/wiki/xacro">
-   <joint
+  <joint
     name="body_base_joint"
     type="fixed">

File: ros2_rm_robot/dual_rm_description/dual_rm_75b_description/urdf/agv/woosh_agv.urdf.xacro (robot description, xacro)
@@ -2,5 +2,5 @@
 <robot name="woosh_agv" xmlns:xacro="http://www.ros.org/wiki/xacro">
   <!-- Define constants -->
-  <xacro:property name="mesh_path" value="file://$(find dual_rm_65b_description)/meshes/" />
+  <xacro:property name="mesh_path" value="file://$(find dual_rm_75b_description)/meshes/" />
   <!-- Macro for visual and collision elements -->
   <xacro:macro name="visual_collision" params="mesh">
@@ -39,4 +39,6 @@
     <xacro:visual_collision mesh="base_link_underpan.STL" />
   </link>
+  <!-- Drive wheels: mesh for visual, CYLINDER for collision (reliable rolling contact in Gz Sim) -->
+  <!-- Wheel geometry: radius=0.08m, width≈0.05m, axis along X -->
   <link
     name="link_right_wheel">
@@ -55,5 +57,20 @@
         izz="0.0018066" />
     </inertial>
-    <xacro:visual_collision mesh="link_right_wheel.STL" />
+    <visual>
+      <origin xyz="0 0 0" rpy="0 0 0" />
+      <geometry>
+        <mesh filename="${mesh_path}link_right_wheel.STL" />
+      </geometry>
+      <material name="">
+        <color rgba="0.79216 0.81961 0.93333 1" />
+      </material>
+    </visual>
+    <collision>
+      <!-- Cylinder along X axis: rotate 90° around Y -->
+      <origin xyz="-0.025 0 0" rpy="0 ${pi/2} 0" />
+      <geometry>
+        <cylinder radius="0.08" length="0.05" />
+      </geometry>
+    </collision>
   </link>
   <link
@@ -73,5 +90,20 @@
         izz="0.0019593" />
     </inertial>
-    <xacro:visual_collision mesh="link_left_wheel.STL" />
+    <visual>
+      <origin xyz="0 0 0" rpy="0 0 0" />
+      <geometry>
+        <mesh filename="${mesh_path}link_left_wheel.STL" />
+      </geometry>
+      <material name="">
+        <color rgba="0.79216 0.81961 0.93333 1" />
+      </material>
+    </visual>
+    <collision>
+      <!-- Cylinder along X axis: rotate 90° around Y -->
+      <origin xyz="0.025 0 0" rpy="0 ${pi/2} 0" />
+      <geometry>
+        <cylinder radius="0.08" length="0.05" />
+      </geometry>
+    </collision>
   </link>
   <link
@@ -246,5 +278,5 @@
       link="link_left_wheel" />
     <axis
-      xyz="-1 0 0" />
+      xyz="1 0 0" />
     <limit
       effort="100"

File: ros2_rm_robot/dual_rm_description/dual_rm_75b_description/urdf/dual_rm_75b_description.urdf.xacro (robot description, xacro)
@@ -1,16 +1,32 @@
 <?xml version="1.0"?>
+<!--
+  R2D3 75b Robot Description — main xacro entry point.
+  Assembles the full robot from modular sub-components:
+    agv/            — AGV chassis, drive wheels, caster wheels
+    body/           — Torso, head, camera, platform lift
+    left_arm/       — Left 7-DOF arm + gripper
+    right_arm/      — Right 7-DOF arm + gripper
+    joints/         — Cross-component joints (body↔arms, arms↔hands)
+    materials/      — Named URDF colour definitions
+    transmissions/  — Legacy ROS1 transmission tags (kept for compatibility)
+-->
 <robot name="dual_rm_75b_description" xmlns:xacro="http://ros.org/wiki/xacro">
-  <!-- 引入各个模块的 xacro 文件，分别定义底盘、夹爪、升降平台、机械臂及关节 -->
-  <xacro:include filename="$(find dual_rm_75b_description)/urdf/woosh_agv.urdf.xacro"/>
-  <xacro:include filename="$(find dual_rm_75b_description)/urdf/body_head_platform.urdf.xacro"/>
-  <xacro:include filename="$(find dual_rm_75b_description)/urdf/left_hand.urdf.xacro"/>
-  <xacro:include filename="$(find dual_rm_75b_description)/urdf/right_hand.urdf.xacro"/>
-  <xacro:include filename="$(find dual_rm_75b_description)/urdf/rm75_b_v_left.urdf.xacro"/>
-  <xacro:include filename="$(find dual_rm_75b_description)/urdf/rm75_b_v_right.urdf.xacro"/>
-  <xacro:include filename="$(find dual_rm_75b_description)/urdf/joint.urdf.xacro"/>
-  <!-- 在 Gazebo 仿真环境中添加控制传动配置及 Gazebo 专用插件 -->
-  <xacro:include filename="$(find dual_rm_75b_description)/urdf/rm75_b_v_left_transmission.xacro"/>
-  <xacro:include filename="$(find dual_rm_75b_description)/urdf/rm75_b_v_right_transmission.xacro"/>
-  <xacro:include filename="$(find dual_rm_75b_description)/urdf/body_head_platform_transmission.xacro"/>
-  <!-- <xacro:include filename="$(find dual_rm_75b_description)/urdf/common_gazebo.xacro"/> -->
+    <!-- ── Materials ─────────────────────────────────────────── -->
+    <xacro:include filename="$(find dual_rm_75b_description)/urdf/materials/colors.urdf.xacro"/>
+    <!-- ── AGV chassis (wheels, casters) ─────────────────────── -->
+    <xacro:include filename="$(find dual_rm_75b_description)/urdf/agv/woosh_agv.urdf.xacro"/>
+    <!-- ── Body, head, camera, platform lift ─────────────────── -->
+    <xacro:include filename="$(find dual_rm_75b_description)/urdf/body/body_head_platform.urdf.xacro"/>
+    <!-- ── Left arm (7-DOF) + gripper ────────────────────────── -->
+    <xacro:include filename="$(find dual_rm_75b_description)/urdf/left_arm/rm75_b_v_left.urdf.xacro"/>
+    <xacro:include filename="$(find dual_rm_75b_description)/urdf/left_arm/left_hand.urdf.xacro"/>
+    <!-- ── Right arm (7-DOF) + gripper ───────────────────────── -->
+    <xacro:include filename="$(find dual_rm_75b_description)/urdf/right_arm/rm75_b_v_right.urdf.xacro"/>
+    <xacro:include filename="$(find dual_rm_75b_description)/urdf/right_arm/right_hand.urdf.xacro"/>
+    <!-- ── Cross-component joints ────────────────────────────── -->
+    <xacro:include filename="$(find dual_rm_75b_description)/urdf/joints/joint.urdf.xacro"/>
+    <!-- ── Transmissions (legacy ROS1, kept for compatibility) ── -->
+    <xacro:include filename="$(find dual_rm_75b_description)/urdf/transmissions/rm75_b_v_left_transmission.xacro"/>
+    <xacro:include filename="$(find dual_rm_75b_description)/urdf/transmissions/rm75_b_v_right_transmission.xacro"/>
+    <xacro:include filename="$(find dual_rm_75b_description)/urdf/transmissions/body_head_platform_transmission.xacro"/>
 </robot>
