Commit message: Integrated Issac Sim and Sensor Inputs

File: isaac_sim/urdf/parallel_gripper.urdf.xacro (robot description, xacro)
@@ -83,9 +83,9 @@
     </joint>
     <!--
-      Mimic joint. Axis -Y so that the same positive joint value drives the
-      RIGHT finger in the OPPOSITE direction. Mimic multiplier = +1 so both
-      joints share their parameter; the axis sign delivers the symmetry.
-      This keeps both joints in [0, 0.035], satisfying their limits and
-      Isaac Sim's PhysX Tendon (parse_mimic=True) representation.
+      Mimic joint. Authored as a plain prismatic (no <mimic> element) so the
+      URDF→USD converter doesn't apply NewtonMimicAPI — the default PhysX
+      solver in Isaac Sim 6.0 doesn't honor it and the articulation goes NaN.
+      Symmetric closure is enforced in robot.set_finger(): both finger_drive
+      and finger_mimic are commanded to the same scalar.
     -->
     <joint name="${prefix}finger_mimic" type="prismatic">
@@ -96,5 +96,4 @@
       <limit lower="0.0" upper="0.035" velocity="0.05" effort="100"/>
       <dynamics damping="1.0" friction="0.1"/>
-      <mimic joint="${prefix}finger_drive" multiplier="1.0" offset="0.0"/>
     </joint>
   </xacro:macro>

File: isaac_sim/urdf/r2d3_v1.urdf.xacro (robot description, xacro)
@@ -25,5 +25,9 @@
        mesh is omitted. Switch to "true" once the converter accepts the .dae
        (or replace with an .stl). -->
-  <xacro:sensor_d435 parent="head_link2" name="head_camera" use_nominal_extrinsics="false" use_mesh="false">
+  <!-- use_nominal_extrinsics="true" authors the REP-103 optical frames
+       (head_camera_color_optical_frame, head_camera_depth_optical_frame, ...)
+       so the camera's published frame_ids actually exist in the TF tree.
+       use_mesh stays false (the .dae still trips the converter). -->
+  <xacro:sensor_d435 parent="head_link2" name="head_camera" use_nominal_extrinsics="true" use_mesh="false">
     <origin xyz="0.05 0.0 0.0" rpy="0 0 0"/>
   </xacro:sensor_d435>
