Commit message: Platform SDK + plug-and-play setup
Turn the working sim into a usable platform.

SDK (isaac_sim/r2d3_sim/): R2D3 facade — one in-process handle for control
(IK set_arm_pose, set_gripper/head/lift/base, set_joint_targets) + sensing
(get_image/depth as numpy without ROS, wrench, FK, observation). Supporting
modules boot/helpers/cameras/ik; envs/ for RL (R2D3Env), VLM (PerceptionLoop),
teleop (TeleopServer). robot.py gains public set_joint_targets/set_base_pose/
get_ee_pose. 7 clean examples; 21 diagnostics archived; docs api/run/platform/
examples/bridge + index hub.

Plug-and-play setup:
- scripts/isaacsim_ros2.sh auto-detects the conda base (no hardcoded home dir)
  and makes ros_humble optional (SDK path needs only the isaac env)
- pyproject.toml -> pip install -e . (sys.path hacks removed from examples)
- ship the built, portable USD assets (usd_dexterous/gripper/mobile)
- requirements.txt + scripts/bootstrap.sh one-command setup; scripts/_conda_env.sh
- build_robot.sh / urdf_to_usd.py de-hardcoded + a mobile build target

Verified headless: smoke_sdk, grasp_cube (cube +0.21 m), drive_base, and the
full bootstrap (launcher + editable install + smoke).

File: isaac_sim/urdf/r2d3_v1.urdf.xacro (robot description, xacro)
@@ -15,29 +15,56 @@
   <!-- 1) The upstream R2D3 (dual RM75-B arms + body lift + head + AGV + hand bodies) -->
   <xacro:include filename="$(find dual_rm_75b_description)/urdf/dual_rm_75b_description.urdf.xacro"/>
-  <!-- 2) Head-mounted Intel RealSense D435.
+  <!-- 2) Cameras (Intel RealSense D435).
        sensor_d435 macro signature:
          params parent *origin name:=camera use_nominal_extrinsics:=false add_plug:=false use_mesh:=true
-  -->
+       use_mesh="false" sidesteps a Collada parse failure in urdf_usd_converter
+       on d435.dae; kinematic frames + bbox geometry are still authored.
+       use_nominal_extrinsics="true" authors the REP-103 optical frames
+       (<name>_color_optical_frame, <name>_depth_optical_frame, ...). -->
   <xacro:include filename="$(find realsense2_description)/urdf/_d435.urdf.xacro"/>
-  <!-- use_mesh="false" sidesteps a Collada parsing failure in
-       urdf_usd_converter 0.1.0 on realsense2_description's d435.dae. Kinematic
-       frames + bounding-box geometry are still authored; only the photorealistic
-       mesh is omitted. Switch to "true" once the converter accepts the .dae
-       (or replace with an .stl). -->
-  <!-- use_nominal_extrinsics="true" authors the REP-103 optical frames
-       (head_camera_color_optical_frame, head_camera_depth_optical_frame, ...)
-       so the camera's published frame_ids actually exist in the TF tree.
-       use_mesh stays false (the .dae still trips the converter). -->
+  <!-- 2a) HEAD camera. The upstream dual_rm_75b head already carries its own
+       camera body (link `camera_link`, via `camera_joint` at
+       xyz=-0.0032391 -0.051866 0.061606 from head_link2) — that is the robot's
+       REAL head camera and stays as the visible body. We only add the D435
+       optical frames + sim sensor here, CO-LOCATED with camera_link, so the ROS
+       camera images from the real camera. (origin = camera_joint xyz minus the
+       d435 bottom_screw->camera_link offset 0.0106 0.0175 0.0125.) -->
   <xacro:sensor_d435 parent="head_link2" name="head_camera" use_nominal_extrinsics="true" use_mesh="false">
-    <origin xyz="0.05 0.0 0.0" rpy="0 0 0"/>
+    <origin xyz="-0.0138391 -0.069366 0.049106" rpy="0 0 0"/>
   </xacro:sensor_d435>
-  <!-- 3) Parallel grippers on both hands.
-       NOTE: the upstream 75b URDF uses asymmetric link names — the LEFT hand
-       is `l_hand_link`, the RIGHT hand is `r_hand`. The mesh files happen to
-       be named `*_hand_base_link.STL` but the link names that reference them
-       are not. Verified 2026-05-19 against
-       ros2_rm_robot/.../dual_rm_75b_description.urdf (rendered). -->
-  <xacro:include filename="parallel_gripper.urdf.xacro"/>
-  <xacro:parallel_gripper prefix="l_" parent="l_hand_link"/>
-  <xacro:parallel_gripper prefix="r_" parent="r_hand"/>
+  <!-- 2b) WRIST cameras (in-hand view), one per arm, on the last arm link.
+       l_link7 / r_link7 +Z points toward the hand (hand mounts at +Z 0.0445),
+       so rpy="0 -pi/2 0" aims the D435's forward (+X) down +Z at the grasp.
+       Mounted offset to the side of the wrist so it clears the arm/hand. -->
+  <xacro:sensor_d435 parent="l_link7" name="l_wrist_camera" use_nominal_extrinsics="true" use_mesh="false">
+    <origin xyz="0.05 0.0 0.0" rpy="0 -1.5707963 0"/>
+  </xacro:sensor_d435>
+  <xacro:sensor_d435 parent="r_link7" name="r_wrist_camera" use_nominal_extrinsics="true" use_mesh="false">
+    <origin xyz="0.05 0.0 0.0" rpy="0 -1.5707963 0"/>
+  </xacro:sensor_d435>
+  <!-- 3) End-effector — SWITCHABLE. Both mount on the arm hand links
+       (LEFT = l_hand_link, RIGHT = r_hand; the 75b URDF link names are
+       asymmetric). Select with the xacro arg:
+         xacro r2d3_v1.urdf.xacro end_effector:=dexterous   (Inspire RH56 hand)
+         xacro r2d3_v1.urdf.xacro end_effector:=gripper     (parallel gripper)
+       scripts/build_robot.sh builds a USD per variant. -->
+  <xacro:arg name="end_effector" default="dexterous"/>
+  <xacro:property name="ee" value="$(arg end_effector)"/>
+  <!-- 3a) Inspire RH56 6-DOF / 5-finger dexterous hands (real R2D3 hardware).
+       Macro generated by generate_inspire_macro.py from dexsuite/dex-urdf. -->
+  <xacro:if value="${ee == 'dexterous'}">
+    <xacro:include filename="inspire_hand.urdf.xacro"/>
+    <xacro:inspire_hand prefix="l_dex_" side="left" parent="l_hand_link">
+      <origin xyz="0 0 0" rpy="-1.5707963 0 3.14159"/>
+    </xacro:inspire_hand>
+    <xacro:inspire_hand prefix="r_dex_" side="right" parent="r_hand">
+      <origin xyz="0 0 0" rpy="-1.5707963 0 3.14159"/>
+    </xacro:inspire_hand>
+  </xacro:if>
+  <!-- 3b) Parallel gripper (the V1 2-finger stand-in). -->
+  <xacro:if value="${ee == 'gripper'}">
+    <xacro:include filename="parallel_gripper.urdf.xacro"/>
+    <xacro:parallel_gripper prefix="l_" parent="l_hand_link"/>
+    <xacro:parallel_gripper prefix="r_" parent="r_hand"/>
+  </xacro:if>
 </robot>
