Commit message: replaced the gripper with 2 finger gripper and MoveIt setup is in progress

File: ros2_rm_robot/dual_rm_description/dual_rm_75b_description/urdf/dual_rm_75b_description.urdf.xacro (robot description, xacro)
@@ -4,6 +4,7 @@
   <xacro:include filename="$(find dual_rm_75b_description)/urdf/woosh_agv.urdf.xacro"/>
   <xacro:include filename="$(find dual_rm_75b_description)/urdf/body_head_platform.urdf.xacro"/>
-  <xacro:include filename="$(find dual_rm_75b_description)/urdf/left_hand.urdf.xacro"/>
-  <xacro:include filename="$(find dual_rm_75b_description)/urdf/right_hand.urdf.xacro"/>
+  <xacro:include filename="$(find dual_rm_75b_description)/urdf/4c2_attachments.urdf.xacro"/>
+  <!-- <xacro:include filename="$(find dual_rm_75b_description)/urdf/left_hand.urdf.xacro"/> -->
+  <!-- <xacro:include filename="$(find dual_rm_75b_description)/urdf/right_hand.urdf.xacro"/> -->
   <xacro:include filename="$(find dual_rm_75b_description)/urdf/rm75_b_v_left.urdf.xacro"/>
   <xacro:include filename="$(find dual_rm_75b_description)/urdf/rm75_b_v_right.urdf.xacro"/>

File: ros2_rm_robot/dual_rm_description/dual_rm_75b_description/urdf/joint.urdf.xacro (robot description, xacro)
@@ -43,5 +43,5 @@
       xyz="0 0 0" />
   </joint>
-  <joint
+  <!-- <joint
     name="r_hand_joint"
     type="fixed">
@@ -60,6 +60,6 @@
       effort="0"
       velocity="0" />
-  </joint>
-  <joint
+  </joint> -->
+  <!-- <joint
     name="l_hand_joint"
     type="fixed">
@@ -78,4 +78,4 @@
       effort="0"
       velocity="0" />
-  </joint>
+  </joint>   -->
 </robot>

File: ros2_rm_robot/dual_rm_description/dual_rm_75b_description/urdf/rm75_b_v_left.urdf.xacro (robot description, xacro)
@@ -147,5 +147,5 @@
     <xacro:visual_collision mesh="l_link6.STL" />
   </link>
-  <link
+  <!-- <link
     name="l_link7">
     <inertial>
@@ -162,7 +162,7 @@
         iyz="-1.7799E-08"
         izz="0.00035278" />
-    </inertial>
-    <xacro:visual_collision mesh="l_link7.STL" />
-  </link>
+    </inertial> -->
+    <!-- <xacro:visual_collision mesh="l_link7.STL" />
+  </link> -->
   <joint
     name="l_joint1"
@@ -273,5 +273,5 @@
       velocity="3.925" />
   </joint>
-  <joint
+  <!-- <joint
     name="l_joint7"
     type="revolute">
@@ -290,4 +290,4 @@
       effort="10"
       velocity="3.925" />
-  </joint>
+  </joint> -->
 </robot>

File: ros2_rm_robot/dual_rm_description/dual_rm_75b_description/urdf/rm75_b_v_left_transmission.xacro (robot description, xacro)
@@ -18,4 +18,4 @@
   <xacro:rm75_b_v_left_transmission joint_name="l_joint5" />
   <xacro:rm75_b_v_left_transmission joint_name="l_joint6" />
-  <xacro:rm75_b_v_left_transmission joint_name="l_joint7" />
+  <!-- <xacro:rm75_b_v_left_transmission joint_name="l_joint7" /> -->
 </robot>

File: ros2_rm_robot/dual_rm_description/dual_rm_75b_description/urdf/rm75_b_v_right.urdf.xacro (robot description, xacro)
@@ -147,5 +147,5 @@
     <xacro:visual_collision mesh="r_link6.STL" />
   </link>
-  <link
+  <!-- <link
     name="r_link7">
     <inertial>
@@ -163,6 +163,6 @@
         izz="0.00035277" />
     </inertial>
-    <xacro:visual_collision mesh="r_link7.STL" />
-  </link>
+    <xacro:visual_collision mesh="r_link7.STL" /> -->
+  <!-- </link> -->
   <joint
     name="r_joint1"
@@ -273,5 +273,5 @@
       velocity="3.925" />
   </joint>
-  <joint
+  <!-- <joint
     name="r_joint7"
     type="revolute">
@@ -290,4 +290,4 @@
       effort="10"
       velocity="3.925" />
-  </joint>
+  </joint> -->
 </robot>

File: ros2_rm_robot/dual_rm_description/dual_rm_75b_description/urdf/rm75_b_v_right_transmission.xacro (robot description, xacro)
@@ -18,4 +18,4 @@
   <xacro:rm75_b_v_right_transmission joint_name="r_joint5" />
   <xacro:rm75_b_v_right_transmission joint_name="r_joint6" />
-  <xacro:rm75_b_v_right_transmission joint_name="r_joint7" />
+  <!-- <xacro:rm75_b_v_right_transmission joint_name="r_joint7" /> -->
 </robot>

File: ros2_rm_robot/dual_rm_description/dual_rm_75b_description/urdf/woosh_agv.urdf.xacro (robot description, xacro)
@@ -223,5 +223,5 @@
     type="continuous">
     <origin
-      xyz="-0.148 0.015574 -0.153"
+      xyz="-0.148 0.015574 -0.16254"
       rpy="0 0 0" />
     <parent
@@ -239,5 +239,5 @@
     type="continuous">
     <origin
-      xyz="0.148 0.015574 -0.153"
+      xyz="0.148 0.015574 -0.16254"
       rpy="0 0 0" />
     <parent
@@ -246,5 +246,5 @@
       link="link_left_wheel" />
     <axis
-      xyz="-1 0 0" />
+      xyz="1 0 0" />
     <limit
       effort="100"

File: ros2_rm_robot/dual_rm_moveit_config/dual_rm_75b_moveit_config/config/dual_rm_75b_description.ros2_control.xacro (robot description, xacro)
@@ -50,8 +50,15 @@
                 <state_interface name="velocity"/>
             </joint>
-            <joint name="l_joint7">
+            <!-- <joint name="l_joint7">
                 <command_interface name="position"/>
                 <state_interface name="position">
                   <param name="initial_value">${initial_positions['l_joint7']}</param>
+                </state_interface>
+                <state_interface name="velocity"/>
+            </joint> -->
+            <joint name="l_4c2_gripper_joint">
+                <command_interface name="position"/>
+                <state_interface name="position">
+                  <param name="initial_value">${initial_positions['l_4c2_gripper_joint']}</param>
                 </state_interface>
                 <state_interface name="velocity"/>
@@ -99,8 +106,15 @@
                 <state_interface name="velocity"/>
             </joint>
-            <joint name="r_joint7">
+            <!-- <joint name="r_joint7">
                 <command_interface name="position"/>
                 <state_interface name="position">
                   <param name="initial_value">${initial_positions['r_joint7']}</param>
+                </state_interface>
+                <state_interface name="velocity"/>
+            </joint> -->
+            <joint name="r_4c2_gripper_joint">
+                <command_interface name="position"/>
+                <state_interface name="position">
+                  <param name="initial_value">${initial_positions['r_4c2_gripper_joint']}</param>
                 </state_interface>
                 <state_interface name="velocity"/>

Commit message: Revert "replaced the gripper with 2 finger gripper, MoveIt in progress"

File: ros2_rm_robot/dual_rm_description/dual_rm_75b_description/urdf/dual_rm_75b_description.urdf.xacro (robot description, xacro)
@@ -4,7 +4,6 @@
   <xacro:include filename="$(find dual_rm_75b_description)/urdf/woosh_agv.urdf.xacro"/>
   <xacro:include filename="$(find dual_rm_75b_description)/urdf/body_head_platform.urdf.xacro"/>
-  <xacro:include filename="$(find dual_rm_75b_description)/urdf/4c2_attachments.urdf.xacro"/>
-  <!-- <xacro:include filename="$(find dual_rm_75b_description)/urdf/left_hand.urdf.xacro"/> -->
-  <!-- <xacro:include filename="$(find dual_rm_75b_description)/urdf/right_hand.urdf.xacro"/> -->
+  <xacro:include filename="$(find dual_rm_75b_description)/urdf/left_hand.urdf.xacro"/>
+  <xacro:include filename="$(find dual_rm_75b_description)/urdf/right_hand.urdf.xacro"/>
   <xacro:include filename="$(find dual_rm_75b_description)/urdf/rm75_b_v_left.urdf.xacro"/>
   <xacro:include filename="$(find dual_rm_75b_description)/urdf/rm75_b_v_right.urdf.xacro"/>

File: ros2_rm_robot/dual_rm_description/dual_rm_75b_description/urdf/joint.urdf.xacro (robot description, xacro)
@@ -43,5 +43,5 @@
       xyz="0 0 0" />
   </joint>
-  <!-- <joint
+  <joint
     name="r_hand_joint"
     type="fixed">
@@ -60,6 +60,6 @@
       effort="0"
       velocity="0" />
-  </joint> -->
-  <!-- <joint
+  </joint>
+  <joint
     name="l_hand_joint"
     type="fixed">
@@ -78,4 +78,4 @@
       effort="0"
       velocity="0" />
-  </joint>   -->
+  </joint>
 </robot>

File: ros2_rm_robot/dual_rm_description/dual_rm_75b_description/urdf/rm75_b_v_left.urdf.xacro (robot description, xacro)
@@ -147,5 +147,5 @@
     <xacro:visual_collision mesh="l_link6.STL" />
   </link>
-  <!-- <link
+  <link
     name="l_link7">
     <inertial>
@@ -162,7 +162,7 @@
         iyz="-1.7799E-08"
         izz="0.00035278" />
-    </inertial> -->
-    <!-- <xacro:visual_collision mesh="l_link7.STL" />
-  </link> -->
+    </inertial>
+    <xacro:visual_collision mesh="l_link7.STL" />
+  </link>
   <joint
     name="l_joint1"
@@ -273,5 +273,5 @@
       velocity="3.925" />
   </joint>
-  <!-- <joint
+  <joint
     name="l_joint7"
     type="revolute">
@@ -290,4 +290,4 @@
       effort="10"
       velocity="3.925" />
-  </joint> -->
+  </joint>
 </robot>

File: ros2_rm_robot/dual_rm_description/dual_rm_75b_description/urdf/rm75_b_v_right.urdf.xacro (robot description, xacro)
@@ -147,5 +147,5 @@
     <xacro:visual_collision mesh="r_link6.STL" />
   </link>
-  <!-- <link
+  <link
     name="r_link7">
     <inertial>
@@ -163,6 +163,6 @@
         izz="0.00035277" />
     </inertial>
-    <xacro:visual_collision mesh="r_link7.STL" /> -->
-  <!-- </link> -->
+    <xacro:visual_collision mesh="r_link7.STL" />
+  </link>
   <joint
     name="r_joint1"
@@ -273,5 +273,5 @@
       velocity="3.925" />
   </joint>
-  <!-- <joint
+  <joint
     name="r_joint7"
     type="revolute">
@@ -290,4 +290,4 @@
       effort="10"
       velocity="3.925" />
-  </joint> -->
+  </joint>
 </robot>

File: ros2_rm_robot/dual_rm_description/dual_rm_75b_description/urdf/woosh_agv.urdf.xacro (robot description, xacro)
@@ -223,5 +223,5 @@
     type="continuous">
     <origin
-      xyz="-0.148 0.015574 -0.16254"
+      xyz="-0.148 0.015574 -0.153"
       rpy="0 0 0" />
     <parent
@@ -239,5 +239,5 @@
     type="continuous">
     <origin
-      xyz="0.148 0.015574 -0.16254"
+      xyz="0.148 0.015574 -0.153"
       rpy="0 0 0" />
     <parent
@@ -246,5 +246,5 @@
       link="link_left_wheel" />
     <axis
-      xyz="1 0 0" />
+      xyz="-1 0 0" />
     <limit
       effort="100"

File: ros2_rm_robot/dual_rm_moveit_config/dual_rm_75b_moveit_config/config/dual_rm_75b_description.ros2_control.xacro (robot description, xacro)
@@ -50,15 +50,8 @@
                 <state_interface name="velocity"/>
             </joint>
-            <!-- <joint name="l_joint7">
+            <joint name="l_joint7">
                 <command_interface name="position"/>
                 <state_interface name="position">
                   <param name="initial_value">${initial_positions['l_joint7']}</param>
-                </state_interface>
-                <state_interface name="velocity"/>
-            </joint> -->
-            <joint name="l_4c2_gripper_joint">
-                <command_interface name="position"/>
-                <state_interface name="position">
-                  <param name="initial_value">${initial_positions['l_4c2_gripper_joint']}</param>
                 </state_interface>
                 <state_interface name="velocity"/>
@@ -106,15 +99,8 @@
                 <state_interface name="velocity"/>
             </joint>
-            <!-- <joint name="r_joint7">
+            <joint name="r_joint7">
                 <command_interface name="position"/>
                 <state_interface name="position">
                   <param name="initial_value">${initial_positions['r_joint7']}</param>
-                </state_interface>
-                <state_interface name="velocity"/>
-            </joint> -->
-            <joint name="r_4c2_gripper_joint">
-                <command_interface name="position"/>
-                <state_interface name="position">
-                  <param name="initial_value">${initial_positions['r_4c2_gripper_joint']}</param>
                 </state_interface>
                 <state_interface name="velocity"/>
