Commit message: feat(r2d3_mujoco): validated URDF->MJCF conversion; wheel/caster contact tuning
Ran the real make_mjcf_from_robot_description converter against the R2D3
URDF+nav_empty scene, fixed a missing MJCF collision/visual <default> block
(the converter tags every geom with those classes but never defines them),
and validated the resulting model headlessly with mujoco.MjModel (free
joint settle, straight drive, in-place turn, 30s drift check all pass).

Wheel/caster geoms turn out to be unnamed in the generated MJCF (the
description is visual-only, so the converter synthesizes collision geometry
without a name attribute), so per-geom modify_element targeting isn't
possible; applied the drive-wheel friction/condim tuning to the shared
"collision" default class instead and added noslip_iterations=3 to curb
drive drift. Full investigation and rationale recorded in SPIKE_NOTES.md.

Co-Authored-By: Claude Fable 5 <noreply@anthropic.com>
Claude-Session: https://claude.ai/code/session_01Kfm6fGJVZ2dVdCFetsAdGD

File: r2d3_mujoco/urdf/mujoco_inputs.urdf.xacro (robot description, xacro)
@@ -20,5 +20,36 @@
         <mujoco_inputs>
             <raw_inputs>
-                <option integrator="implicitfast"/>
+                <option integrator="implicitfast" noslip_iterations="3"/>
+                <!-- Required: the converter emits every geom with class="collision" or
+                     class="visual" but never defines those classes itself (see
+                     mujoco_ros2_control/urdf_to_mujoco_utils.py). Without this default
+                     block the compiler rejects the MJCF with
+                     "unknown default class name 'collision'". -->
+                <!-- Wheel/caster traction (Task 4 spike finding): the R2D3 description
+                     is visual-only (no <collision> elements), so the converter
+                     synthesizes every collision geom from the visual mesh with NO
+                     name attribute (confirmed: 0 of 68 robot geoms in the generated
+                     MJCF carry a name, only the scene's static geoms do). modify_element
+                     matches strictly on an element's existing "name" attribute, so
+                     individual wheel/caster geoms cannot be targeted: there is no
+                     name for it to match. The friction/condim values below (matching
+                     the Gazebo drive-wheel tuning, mu 1.5) are therefore applied via
+                     the shared "collision" default class, i.e. to every robot collision
+                     geom. This is safe here because only the wheels/casters normally
+                     contact the ground; the platform's casters are modeled as real
+                     2-DOF (swivel+roll) joints (see robot_description_formatted.urdf),
+                     so they self-align under drive torque rather than needing an
+                     artificially low ground-contact mu the way Gazebo's simplified
+                     single-DOF caster friction model did. See SPIKE_NOTES.md for the
+                     full investigation (decompose_mesh/obj2mjcf naming was also checked
+                     and does not produce named geoms either). -->
+                <default>
+                    <default class="visual">
+                        <geom group="2" type="mesh" contype="0" conaffinity="0"/>
+                    </default>
+                    <default class="collision">
+                        <geom group="3" type="mesh" friction="1.5 0.005 0.0001" condim="4"/>
+                    </default>
+                </default>
                 <actuator>
                     <!-- Drive wheels: native velocity actuators (matches the
@@ -100,6 +131,10 @@
                 <xacro:_mj_gravcomp body_name="head_link2"/>
                 <xacro:_mj_gravcomp body_name="platform_base_link"/>
-                <!-- Wheel/caster friction tuning is added here in Task 4 after the
-                     generated geom names are known (modify_element type="geom" ...) -->
+                <!-- Wheel/caster friction tuning (Task 4): applied via the shared
+                     "collision" default class in raw_inputs above, not via
+                     modify_element, because the converter never assigns a "name"
+                     to synthesized collision geoms for this (visual-only)
+                     description, so there is nothing modify_element type="geom"
+                     could match. See SPIKE_NOTES.md for the full investigation. -->
             </processed_inputs>
         </mujoco_inputs>
