Commit message: fix(sim): compensate base +90 yaw in camera optical frame (camera bores forward)
The URDF unification (9a01958) removed the camera_joint -90 hack from the
core description (correct: real robot camera_joint=0) but never re-added the
compensation in the sim overlay, so the head-mounted camera rode the
base_footprint_to_base +90 mesh->nav yaw and /camera/image looked 90 deg
left. Fold the -90 into the sim-only camera_optical_joint. MuJoCo only;
Gazebo tracked separately.

File: ros2_rm_robot/dual_rm_simulation/urdf/sensors/depth_camera.urdf.xacro (robot description, xacro)
@@ -10,6 +10,16 @@
             <parent link="camera_link"/>
             <child link="camera_optical_frame"/>
-            <!-- Rotate from body frame (X-fwd) to optical frame (Z-fwd) -->
-            <origin xyz="0 0 0" rpy="${-pi/2} 0 ${-pi/2}"/>
+            <!-- Body-frame (X-fwd) -> optical (Z-fwd) is the standard
+                 rpy="-pi/2 0 -pi/2". The trailing yaw carries an EXTRA -pi/2
+                 (net "-pi/2 0 -pi") to compensate the sim overlay's mesh->nav
+                 +pi/2 yaw at base_footprint_to_base, which yaws the whole
+                 mechanical tree - including this head-mounted camera_link
+                 (camera_link X = base_footprint +Y). Without it the optical
+                 bore points nav +Y and the MuJoCo /camera/image looks 90 deg
+                 to the robot's left. The core description's camera_joint stays
+                 0 (real-faithful); this compensation is sim-only. Do NOT
+                 "simplify" back to -pi/2 - see commit 9a01958 and
+                 docs/superpowers/plans/2026-07-15-camera-optical-frame-yaw-fix.md. -->
+            <origin xyz="0 0 0" rpy="${-pi/2} 0 ${-pi}"/>
         </joint>
         <!-- ── Gazebo physics ──────────────────────────────────────── -->

Commit message: fix(sim): mount Gz camera on -90deg camera_gz_frame so it renders nav-forward
A Gz camera renders along its mount frame's +X; camera_link rides the
sim overlay's +90deg mesh->nav base yaw, so the image looked 90deg left
and disagreed with its camera_optical_frame label (issue #11). Mount the
sensor on a sim-only massless frame instead of a sensor <pose> (banned
by the issue #11 postmortem). Guarded by test_gz_camera_bore.py.

File: ros2_rm_robot/dual_rm_simulation/urdf/sensors/depth_camera.urdf.xacro (robot description, xacro)
@@ -23,4 +23,21 @@
             <origin xyz="0 0 0" rpy="${-pi/2} 0 ${-pi}"/>
         </joint>
+        <!-- ── Sim-only Gz mount frame ─────────────────────────────── -->
+        <!-- A Gz camera renders along the +X of the frame its <sensor>
+             is mounted on (gz_frame_id below only LABELS the output).
+             camera_link rides the sim overlay's base_footprint_to_base
+             +pi/2 mesh->nav yaw, so camera_link +X = base_footprint +Y
+             and an uncompensated Gz camera images 90 deg to the robot's
+             left. This massless frame de-yaws the mount so the render
+             bores nav +X, matching the camera_optical_frame label above.
+             Frame-level only: no mesh, no mechanical angles, and per the
+             issue #11 postmortem do NOT do this with a <pose> inside the
+             <sensor>. Guarded by test/test_gz_camera_bore.py. -->
+        <link name="camera_gz_frame"/>
+        <joint name="camera_gz_joint" type="fixed">
+            <parent link="camera_link"/>
+            <child link="camera_gz_frame"/>
+            <origin xyz="0 0 0" rpy="0 0 ${-pi/2}"/>
+        </joint>
         <!-- ── Gazebo physics ──────────────────────────────────────── -->
         <gazebo reference="camera_link">
@@ -28,5 +45,5 @@
         </gazebo>
         <!-- ── Gz Sim RGBD Camera sensor ───────────────────────────── -->
-        <gazebo reference="camera_link">
+        <gazebo reference="camera_gz_frame">
             <sensor name="depth_camera" type="rgbd_camera">
                 <always_on>true</always_on>
