Commit message: Initial robot start pose update, camera and lidar yaw correcction   as per base offset

File: ros2_rm_robot/dual_rm_description/dual_rm_description/urdf/body/body_head_platform.urdf.xacro (robot description, xacro)
@@ -168,5 +168,5 @@
     <origin
       xyz="-0.0032391 -0.051866 0.061606"
-      rpy="0 0 0" />
+      rpy="0 0 ${-pi/2}" />
     <parent
       link="head_link2" />

File: ros2_rm_robot/dual_rm_gazebo/config/dual_rm_65b_gz_sim.urdf.xacro (robot description, xacro)
@@ -157,5 +157,5 @@
             <command_interface name="position"/>
             <state_interface name="position">
-                <param name="initial_value">0</param>
+                <param name="initial_value">2.0568736101999248</param>
             </state_interface>
             <state_interface name="velocity"/>
@@ -164,5 +164,5 @@
             <command_interface name="position"/>
             <state_interface name="position">
-                <param name="initial_value">0</param>
+                <param name="initial_value">0.553739397760887</param>
             </state_interface>
             <state_interface name="velocity"/>
@@ -171,5 +171,5 @@
             <command_interface name="position"/>
             <state_interface name="position">
-                <param name="initial_value">0</param>
+                <param name="initial_value">1.3360178513191066</param>
             </state_interface>
             <state_interface name="velocity"/>
@@ -178,5 +178,5 @@
             <command_interface name="position"/>
             <state_interface name="position">
-                <param name="initial_value">0</param>
+                <param name="initial_value">0.627859936346868</param>
             </state_interface>
             <state_interface name="velocity"/>
@@ -185,5 +185,5 @@
             <command_interface name="position"/>
             <state_interface name="position">
-                <param name="initial_value">0</param>
+                <param name="initial_value">-2.539121367103219</param>
             </state_interface>
             <state_interface name="velocity"/>
@@ -192,5 +192,5 @@
             <command_interface name="position"/>
             <state_interface name="position">
-                <param name="initial_value">0</param>
+                <param name="initial_value">3.1099294070322805</param>
             </state_interface>
             <state_interface name="velocity"/>
@@ -199,5 +199,5 @@
             <command_interface name="position"/>
             <state_interface name="position">
-                <param name="initial_value">0</param>
+                <param name="initial_value">2.0569178650780406</param>
             </state_interface>
             <state_interface name="velocity"/>
@@ -206,5 +206,5 @@
             <command_interface name="position"/>
             <state_interface name="position">
-                <param name="initial_value">0</param>
+                <param name="initial_value">0.4856440765489487</param>
             </state_interface>
             <state_interface name="velocity"/>
@@ -213,5 +213,5 @@
             <command_interface name="position"/>
             <state_interface name="position">
-                <param name="initial_value">0</param>
+                <param name="initial_value">1.4370323214059306</param>
             </state_interface>
             <state_interface name="velocity"/>
@@ -220,5 +220,5 @@
             <command_interface name="position"/>
             <state_interface name="position">
-                <param name="initial_value">0</param>
+                <param name="initial_value">-0.5151946788810964</param>
             </state_interface>
             <state_interface name="velocity"/>
@@ -227,5 +227,5 @@
             <command_interface name="position"/>
             <state_interface name="position">
-                <param name="initial_value">0</param>
+                <param name="initial_value">2.5845659583029796</param>
             </state_interface>
             <state_interface name="velocity"/>
@@ -234,5 +234,5 @@
             <command_interface name="position"/>
             <state_interface name="position">
-                <param name="initial_value">0</param>
+                <param name="initial_value">0.7905380584362347</param>
             </state_interface>
             <state_interface name="velocity"/>

File: ros2_rm_robot/dual_rm_simulation/urdf/r2d3_sim.urdf.xacro (robot description, xacro)
@@ -27,5 +27,5 @@
     <!-- ── 3. Sensors ────────────────────────────────────────── -->
     <xacro:lidar_sensor parent_link="base_link_underpan"
-                        xyz="0.0 -0.24 0.0" rpy="0 0 0"/>
+                        xyz="0.0 -0.24 0.0" rpy="0 0 ${-pi/2}"/>
     <!-- IMU: centre of AGV chassis -->
     <xacro:imu_sensor parent_link="base_link_underpan"

File: ros2_rm_robot/dual_rm_simulation/urdf/ros2_control/sim_ros2_control.urdf.xacro (robot description, xacro)
@@ -8,9 +8,9 @@
 <robot xmlns:xacro="http://www.ros.org/wiki/xacro">
     <!-- ── Helper: single position-command arm joint ─────────── -->
-    <xacro:macro name="_arm_joint" params="joint_name">
+    <xacro:macro name="_arm_joint" params="joint_name initial_value:=0">
         <joint name="${joint_name}">
             <command_interface name="position"/>
             <state_interface name="position">
-                <param name="initial_value">0</param>
+                <param name="initial_value">${initial_value}</param>
             </state_interface>
             <state_interface name="velocity"/>
@@ -48,10 +48,10 @@
             </joint>
             <!-- ── Left arm (position command) ───────────────── -->
-            <xacro:_arm_joint joint_name="l_joint1"/>
-            <xacro:_arm_joint joint_name="l_joint2"/>
-            <xacro:_arm_joint joint_name="l_joint3"/>
-            <xacro:_arm_joint joint_name="l_joint4"/>
-            <xacro:_arm_joint joint_name="l_joint5"/>
-            <xacro:_arm_joint joint_name="l_joint6"/>
+            <xacro:_arm_joint joint_name="l_joint1" initial_value="3.1099294070322805"/>
+            <xacro:_arm_joint joint_name="l_joint2" initial_value="2.0569178650780406"/>
+            <xacro:_arm_joint joint_name="l_joint3" initial_value="0.4856440765489487"/>
+            <xacro:_arm_joint joint_name="l_joint4" initial_value="1.4370323214059306"/>
+            <xacro:_arm_joint joint_name="l_joint5" initial_value="-0.5151946788810964"/>
+            <xacro:_arm_joint joint_name="l_joint6" initial_value="2.5845659583029796"/>
             <xacro:if value="${arm_dof == 7}">
                 <xacro:_arm_joint joint_name="l_joint7"/>
@@ -59,14 +59,14 @@
             <!-- ── Right arm (position command) ──────────────── -->
             <xacro:_arm_joint joint_name="r_joint1"/>
-            <xacro:_arm_joint joint_name="r_joint2"/>
-            <xacro:_arm_joint joint_name="r_joint3"/>
-            <xacro:_arm_joint joint_name="r_joint4"/>
-            <xacro:_arm_joint joint_name="r_joint5"/>
-            <xacro:_arm_joint joint_name="r_joint6"/>
+            <xacro:_arm_joint joint_name="r_joint2" initial_value="2.0568736101999248"/>
+            <xacro:_arm_joint joint_name="r_joint3" initial_value="0.553739397760887"/>
+            <xacro:_arm_joint joint_name="r_joint4" initial_value="1.3360178513191066"/>
+            <xacro:_arm_joint joint_name="r_joint5" initial_value="0.627859936346868"/>
+            <xacro:_arm_joint joint_name="r_joint6" initial_value="-2.539121367103219"/>
             <xacro:if value="${arm_dof == 7}">
                 <xacro:_arm_joint joint_name="r_joint7"/>
             </xacro:if>
             <!-- ── Platform lift (position command) ──────────── -->
-            <xacro:_arm_joint joint_name="platform_joint"/>
+            <xacro:_arm_joint joint_name="platform_joint" initial_value="0.7905380584362347"/>
             <!-- ── Head joints (position command) ────────────── -->
             <xacro:_arm_joint joint_name="head_joint1"/>

File: ros2_rm_robot/dual_rm_simulation/urdf/sensors/lidar.urdf.xacro (robot description, xacro)
@@ -41,5 +41,5 @@
             <gravity>false</gravity>
         </gazebo>
-        <!-- ── Gazebo gpu_lidar sensor (360°) ────────────────── -->
+        <!-- ── Gazebo gpu_lidar sensor (240°: ±120° from front, matches real robot) -->
         <gazebo reference="lidar_link">
             <sensor name="lidar" type="gpu_lidar">
@@ -52,8 +52,8 @@
                     <scan>
                         <horizontal>
-                            <samples>360</samples>
+                            <samples>240</samples>
                             <resolution>1.0</resolution>
-                            <min_angle>0.0</min_angle>
-                            <max_angle>6.28318</max_angle>
+                            <min_angle>-2.0943951</min_angle>
+                            <max_angle>2.0943951</max_angle>
                         </horizontal>
                     </scan>

Commit message: feat(description): add ZED 2 camera model on head (zed2_camera macro + mesh)

File: ros2_rm_robot/dual_rm_description/dual_rm_description/urdf/body/body_head_platform.urdf.xacro (robot description, xacro)
@@ -2,4 +2,5 @@
 <robot name="body_head_platform" xmlns:xacro="http://www.ros.org/wiki/xacro">
   <xacro:property name="mesh_path" value="file://$(find dual_rm_description)/meshes/common/" />
+  <xacro:include filename="$(find dual_rm_description)/urdf/sensors/zed2.urdf.xacro"/>
   <xacro:macro name="visual_collision" params="mesh">
     <visual>
@@ -180,3 +181,16 @@
       xyz="0 0 0" />
   </joint>
+  <!-- ZED 2 head camera. The -pi/2 yaw is the physical mount: the ZED body
+       is X-forward while the head meshes are modeled -Y-forward (the sim
+       overlay's +pi/2 mesh->nav yaw at base_footprint_to_base makes -Y face
+       nav +X). One fixed physical angle is therefore correct in BOTH the
+       real-faithful core and the sim overlay - the two yaws cancel. No
+       sim-only compensation frames needed (retires the issue #11
+       camera_gz_frame mechanism). Origin inherited from the old camera_joint;
+       real mount offset to be calibrated on hardware. Guarded by
+       dual_rm_simulation/test/test_gz_camera_bore.py and
+       r2d3_mujoco/test/test_camera_optical_frame.py. -->
+  <xacro:zed2_camera name="zed" parent="head_link2">
+    <origin xyz="-0.0032391 -0.051866 0.061606" rpy="0 0 ${-pi/2}"/>
+  </xacro:zed2_camera>
 </robot>

Commit message: refactor!: remove legacy head camera_link/camera_optical_frame (replaced by ZED 2)

File: ros2_rm_robot/dual_rm_description/dual_rm_description/urdf/body/body_head_platform.urdf.xacro (robot description, xacro)
@@ -92,22 +92,4 @@
     <xacro:visual_collision mesh="head_link2.STL" />
   </link>
-  <link
-    name="camera_link">
-    <inertial>
-      <origin
-        xyz="0.0016556 -0.01252 1.2156E-05"
-        rpy="0 0 0" />
-      <mass
-        value="0.049778" />
-      <inertia
-        ixx="4.8577E-06"
-        ixy="4.3442E-07"
-        ixz="-6.2436E-10"
-        iyy="3.075E-05"
-        iyz="6.4645E-10"
-        izz="3.0901E-05" />
-    </inertial>
-    <xacro:visual_collision mesh="camera_link.STL" />
-  </link>
   <joint
     name="platform_joint"
@@ -168,17 +150,4 @@
       velocity="1.57" />
   </joint>
-  <joint
-    name="camera_joint"
-    type="fixed">
-    <origin
-      xyz="-0.0032391 -0.051866 0.061606"
-      rpy="0 0 0" />
-    <parent
-      link="head_link2" />
-    <child
-      link="camera_link" />
-    <axis
-      xyz="0 0 0" />
-  </joint>
   <!-- ZED 2 head camera. The -pi/2 yaw is the physical mount: the ZED body
        is X-forward while the head meshes are modeled -Y-forward (the sim

Commit message: fix(sim): stereo pairing starved by exact-time sync + best-effort QoS; calibrate ZED mount
- stereo_concat: ApproximateTimeSynchronizer (34ms slop) - the sims do NOT
  stamp both eyes identically (mujoco_ros2_control stamps per-camera now(),
  measured 2ms skew ~2/3 of frames; exact sync starved stereo to ~1/3 rate)
- stereo_concat: RELIABLE QoS everywhere - best-effort subscribers lose the
  tail of each ~13MB render burst (right eye measured 10 vs 137 msgs/10s;
  reliable gets 148/149) which also made L/R look like 'the same image'
  (stale right frames + 12px parallax at scene depth)
- zed_mount_joint origin: 30mm forward, 10mm down (calibrated vs head mesh)
- guarded by 3 new wiring tests; live-verified both sims (MuJoCo 109/109/109,
  Gz 148/148/146 L/R/stereo)

File: ros2_rm_robot/dual_rm_description/dual_rm_description/urdf/body/body_head_platform.urdf.xacro (robot description, xacro)
@@ -159,7 +159,10 @@
        real mount offset to be calibrated on hardware. Guarded by
        dual_rm_simulation/test/test_gz_camera_bore.py and
-       r2d3_mujoco/test/test_camera_optical_frame.py. -->
+       r2d3_mujoco/test/test_camera_optical_frame.py.
+       Origin calibrated 2026-07-16 against the head mesh in sim: 30 mm
+       forward (head-forward is -Y in the mesh frame) and 10 mm down from
+       the old camera_joint origin. -->
   <xacro:zed2_camera name="zed" parent="head_link2">
-    <origin xyz="-0.0032391 -0.051866 0.061606" rpy="0 0 ${-pi/2}"/>
+    <origin xyz="-0.0032391 -0.081866 0.051606" rpy="0 0 ${-pi/2}"/>
   </xacro:zed2_camera>
 </robot>
