Commit message: fix(description): 180deg body roll for inverted wrist D435s
The D435 sits inverted in its housing, so rendered images came out upside
down in both sims. Adds the compensating roll on the camera_link -> colour/
depth frame joints.

Placed deliberately BELOW the aim joint. Rolling 180 deg about the bore also
reverses the frame's Y axis, which is the axis tilt turns about: putting this
in the mount rpy leaves bore and image correct while silently inverting the
tilt knob on every arm (verified numerically). Compensating with the mount yaw
just cancels the image flip, so the mount joint cannot carry it at all.

Regression test pins all three properties at once: bore unchanged, image-up
inverted, tilt axis untouched.

File: ros2_rm_robot/dual_rm_description/dual_rm_description/urdf/sensors/d435.urdf.xacro (robot description, xacro)
@@ -41,4 +41,17 @@
       <origin xyz="0 0 0" rpy="0 ${tilt} ${pan}"/>
     </joint>
+    <!-- Body roll: the D435 sits INVERTED in its housing, so the sensor's
+         image-up is opposite the aim frame's +Z. Without this the rendered
+         image comes out upside down (observed in both sims).
+         This roll MUST stay downstream of the aim joint. Rotating 180 deg
+         about the bore necessarily reverses the frame's Y axis, and Y is the
+         axis `tilt` turns about. Put this in the mount joint instead and
+         the tilt knob silently works backwards on every arm. Applied here it
+         leaves the bore and the tilt axis untouched and only flips which way
+         is up in the image. Guarded by
+         test_wrist_camera_mount.py::test_body_roll_preserves_bore_and_tilt_axis.
+         Same value on every wrist today; promote it to wrist_cameras.yaml if a
+         future mount ever carries the camera right-way-up. -->
+    <xacro:property name="body_roll" value="${pi}"/>
     <!-- Colour -->
     <link name="${name}_camera_color_frame"/>
@@ -46,5 +59,5 @@
       <parent link="${name}_camera_link"/>
       <child link="${name}_camera_color_frame"/>
-      <origin xyz="0 0 0" rpy="0 0 0"/>
+      <origin xyz="0 0 0" rpy="${body_roll} 0 0"/>
     </joint>
     <link name="${name}_camera_color_optical_frame"/>
@@ -59,5 +72,5 @@
       <parent link="${name}_camera_link"/>
       <child link="${name}_camera_depth_frame"/>
-      <origin xyz="0 0 0" rpy="0 0 0"/>
+      <origin xyz="0 0 0" rpy="${body_roll} 0 0"/>
     </joint>
     <link name="${name}_camera_depth_optical_frame"/>
